File: eagle/LowVBoard_02.brd (EAGLE design)
At the start: 113 x 48.3 mm, 28 parts, among them IC1 ATMEGA328P-PU, IC2 MCP7940M, IC3 SN74HC595, IC4 SN74HC595, Q1 16MHz, Q2 32.768kHz

Commit message: pcb updates
Parts:
- added J1: CONNJACKR/APCB5.5X2.1MM, Nixie:CONNJACKR/APCB5.5X2.1MM
- S1, S2, S3: value (none) -> TE-SWITCH; device pinhead:1X02/90 -> Nixie:TE-SWITCH
- moved H1 108.4 mm to (108.0, 39.4)
- moved S3 18.2 mm to (43.8, 47.2), flipped to the top, turned to 180 degrees
- moved S2 16.0 mm to (33.0, 47.2), flipped to the top, turned to 180 degrees
- moved S1 12.5 mm to (17.1, 47.2), flipped to the top, turned to 180 degrees
- moved R1 7.24 mm to (12.7, 36.8), turned to 270 degrees
- moved C2 6.13 mm to (11.8, 13.3)
- moved C7 1.91 mm to (104.1, 21.6)
- moved TP_SC_GND 1.91 mm to (110.5, 17.8)
- moved TP_SC_5V 1.90 mm to (110.5, 25.4)
- moved C1 1.42 mm to (11.7, 8.76)
- moved R2 0.64 mm to (5.71, 33.0)
- moved TP_GND 0.64 mm to (69.8, 42.5)
- moved D1 0.64 mm to (83.2, 27.9)
- moved IC1 0.64 mm to (18.4, 20.3)
- moved IC2 0.64 mm to (90.8, 20.3)
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Connections:
- net +5V: now also J1.A
- net GND: now also J1.C, S1.S2, S2.S2, S3.S2; no longer S1.1, S2.1, S3.1
- net SWITCH1: now also S1.S1; no longer S1.2
- net SWITCH2: now also S2.S1; no longer S2.2
- net SWITCH3: now also S3.S1; no longer S3.2
Routing:
- net GND: track 311.7 -> 374.8 mm
- net MINUTE1_B: track 32.0 -> 65.6 mm, vias 0 -> 1
- net SWITCH2: track 22.0 -> 43.0 mm, vias 0 -> 1
- net +5V: track 152.8 -> 169.3 mm
- net SWITCH3: track 23.9 -> 37.9 mm, vias 0 -> 1
- net SWITCH1: track 25.6 -> 37.8 mm, vias 0 -> 1
- net N$56: track 19.8 -> 28.6 mm
- net DOT: track 48.6 -> 41.4 mm
- net HOUR2_B: track 29.7 -> 26.6 mm, vias 0 -> 1
- net MINUTE2_D: track 32.1 -> 34.2 mm, vias 0 -> 1
- net MINUTE1_D: track 23.0 -> 24.2 mm
- net HOUR1_C: track 29.3 -> 30.3 mm
- net MINUTE1_C: track 28.4 -> 29.4 mm
- net MINUTE1_A: track 13.6 -> 14.6 mm
- net HOUR2_C: track 28.5 -> 29.5 mm
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Other:
- board size 113 x 48.3 mm -> 113 x 52.1 mm

Commit message: corrected pcb
Parts:
- moved H1 1.27 mm to (108.0, 40.6)
- moved J1 1.27 mm to (95.9, 48.9)
- moved POWER 1.27 mm to (74.3, 45.1)
- moved R1 1.27 mm to (12.7, 38.1)
- moved S1 1.27 mm to (17.1, 48.5)
- moved S2 1.27 mm to (33.0, 48.5)
- moved S3 1.27 mm to (43.8, 48.5)
- moved TP_SC_5V 1.27 mm to (110.5, 26.7)
- moved Q2 1.27 mm to (88.3, 14.0)
- moved DATA 1.27 mm to (56.5, 3.94)
- moved C1 1.27 mm to (11.7, 10.0)
- moved C2 1.27 mm to (11.8, 14.6)
- moved C3 1.27 mm to (33.7, 12.1)
- moved C4 1.27 mm to (17.1, 12.1)
- moved C5 1.27 mm to (92.1, 12.7)
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Connections:
- net GND: now also J1.B
Routing:
- net GND: track 374.8 -> 380.5 mm
Other:
- outline, holes or cut-outs redrawn
