File: eagle/LowVBoard_02.sch (EAGLE design)
At the start: 28 parts, among them IC1 ATMEGA328P-PU, IC2 MCP7940M, IC3 SN74HC595, IC4 SN74HC595, Q1 16MHz, Q2 32.768kHz

Commit message: pcb updates
Parts:
- added J1: CONNJACKR/APCB5.5X2.1MM, Nixie:CONNJACKR/APCB5.5X2.1MM
- S1, S2, S3: value (none) -> TE-SWITCH; device pinhead:PINHD-1X2/90 -> Nixie:TE-SWITCH
Connections:
- net +5V: now also J1.A
- net GND: now also J1.C, S1.S, S2.S, S3.S; no longer S1.1, S2.1, S3.1
- net SWITCH1: now also S1.P; no longer S1.2
- net SWITCH2: now also S2.P; no longer S2.2
- net SWITCH3: now also S3.P; no longer S3.2
Changed lines of the file:
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@@
 <part name="TP_SC_5V" library="testpad" library_urn="urn:adsk.eagle:library:385" deviceset="TP" device="PAD1-13" package3d_urn="urn:adsk.eagle:package:27946/1"/>
 <part name="TP_SC_GND" library="testpad" library_urn="urn:adsk.eagle:library:385" deviceset="TP" device="PAD1-13" package3d_urn="urn:adsk.eagle:package:27946/1"/>
-<part name="S1" library="pinhead" library_urn="urn:adsk.eagle:library:325" deviceset="PINHD-1X2" device="/90" package3d_urn="urn:adsk.eagle:package:22437/2"/>
-<part name="S2" library="pinhead" library_urn="urn:adsk.eagle:library:325" deviceset="PINHD-1X2" device="/90" package3d_urn="urn:adsk.eagle:package:22437/2"/>
-<part name="S3" library="pinhead" library_urn="urn:adsk.eagle:library:325" deviceset="PINHD-1X2" device="/90" package3d_urn="urn:adsk.eagle:package:22437/2"/>
 <part name="D1" library="Nixie" deviceset="1N4007" device=""/>
 <part name="H1" library="holes" library_urn="urn:adsk.eagle:library:237" deviceset="MOUNT-PAD-ROUND" device="3.3" package3d_urn="urn:adsk.eagle:package:14283/1"/>
+<part name="J1" library="Nixie" deviceset="CONNJACKR/APCB5.5X2.1MM" device=""/>
+<part name="P+2" library="supply1" library_urn="urn:adsk.eagle:library:371" deviceset="+5V" device=""/>
+<part name="GND_1" library="supply1" library_urn="urn:adsk.eagle:library:371" deviceset="GND" device=""/>
+<part name="S1" library="Nixie" deviceset="TE-SWITCH" device=""/>
+<part name="S2" library="Nixie" deviceset="TE-SWITCH" device=""/>
+<part name="S3" library="Nixie" deviceset="TE-SWITCH" device=""/>
 </parts>
 <sheets>
@@
 <attribute name="TP_SIGNAL_NAME" x="240.03" y="-1.27" size="1.778" layer="97" rot="R270"/>
 </instance>
-<instance part="S1" gate="G$1" x="175.26" y="22.86" smashed="yes" rot="R180">
-<attribute name="NAME" x="171.45" y="24.765" size="1.778" layer="95" rot="R180"/>
-<attribute name="VALUE" x="181.61" y="27.94" size="1.778" layer="96" rot="R180"/>
-</instance>
-<instance part="S2" gate="G$1" x="165.1" y="15.24" smashed="yes" rot="R180">
-<attribute name="NAME" x="161.29" y="17.145" size="1.778" layer="95" rot="R180"/>
-<attribute name="VALUE" x="171.45" y="20.32" size="1.778" layer="96" rot="R180"/>
-</instance>
-<instance part="S3" gate="G$1" x="154.94" y="7.62" smashed="yes" rot="R180">
-<attribute name="NAME" x="151.13" y="4.445" size="1.778" layer="95" rot="R180"/>
-<attribute name="VALUE" x="161.29" y="12.7" size="1.778" layer="96" rot="R180"/>
-</instance>
 <instance part="D1" gate="G$1" x="185.42" y="60.96" smashed="yes">
 <attribute name="NAME" x="182.88" y="63.5" size="1.778" layer="95"/>
@@
 <attribute name="NAME" x="234.2642" y="-10.414" size="1.778" layer="95" rot="R270"/>
 <attribute name="VALUE" x="231.2162" y="-10.414" size="1.778" layer="96" rot="R270"/>
+</instance>
+<instance part="J1" gate="G$1" x="17.78" y="45.72" smashed="yes">
+<attribute name="NAME" x="10.16" y="50.8" size="1.778" layer="95"/>
+<attribute name="VALUE" x="10.16" y="40.64" size="1.778" layer="96"/>
+</instance>
+<instance part="P+2" gate="1" x="30.48" y="48.26" smashed="yes" rot="R270">
+<attribute name="VALUE" x="25.4" y="50.8" size="1.778" layer="96"/>
+</instance>
+<instance part="GND_1" gate="1" x="30.48" y="43.18" smashed="yes" rot="R90">
+<attribute name="VALUE" x="33.02" y="40.64" size="1.778" layer="96" rot="R90"/>
+</instance>
+<instance part="S1" gate="G$1" x="185.42" y="20.32" smashed="yes" rot="R270">
+<attribute name="NAME" x="181.61" y="22.86" size="1.778" layer="95"/>
+<attribute name="VALUE" x="181.61" y="16.51" size="1.778" layer="96"/>
+</instance>
+<instance part="S2" gate="G$1" x="177.8" y="12.7" smashed="yes" rot="R270">
+<attribute name="NAME" x="173.99" y="15.24" size="1.778" layer="95"/>
+<attribute name="VALUE" x="176.53" y="8.89" size="1.778" layer="96"/>
+</instance>
+<instance part="S3" gate="G$1" x="172.72" y="5.08" smashed="yes" rot="R270">
+<attribute name="NAME" x="168.91" y="7.62" size="1.778" layer="95"/>
+<attribute name="VALUE" x="168.91" y="1.27" size="1.778" layer="96"/>
 </instance>
 </instances>
@@
 <wire x1="195.58" y1="5.08" x2="195.58" y2="0" width="0.1524" layer="91"/>
 <wire x1="195.58" y1="0" x2="195.58" y2="-5.08" width="0.1524" layer="91"/>
-<wire x1="177.8" y1="20.32" x2="195.58" y2="20.32" width="0.1524" layer="91"/>
+<wire x1="190.5" y1="20.32" x2="195.58" y2="20.32" width="0.1524" layer="91"/>
 <junction x="195.58" y="12.7"/>
 <junction x="195.58" y="5.08"/>
@@
 <wire x1="238.76" y1="0" x2="233.68" y2="0" width="0.1524" layer="91"/>
 <junction x="233.68" y="0"/>
-<pinref part="S1" gate="G$1" pin="1"/>
-<pinref part="S2" gate="G$1" pin="1"/>
-<wire x1="195.58" y1="12.7" x2="167.64" y2="12.7" width="0.1524" layer="91"/>
-<pinref part="S3" gate="G$1" pin="1"/>
-<wire x1="195.58" y1="5.08" x2="157.48" y2="5.08" width="0.1524" layer="91"/>
+<wire x1="195.58" y1="12.7" x2="182.88" y2="12.7" width="0.1524" layer="91"/>
+<wire x1="195.58" y1="5.08" x2="177.8" y2="5.08" width="0.1524" layer="91"/>
 <pinref part="H1" gate="G$1" pin="MOUNT"/>
 <wire x1="233.68" y1="-5.08" x2="233.68" y2="0" width="0.1524" layer="91"/>
+<pinref part="S1" gate="G$1" pin="S"/>
+<pinref part="S2" gate="G$1" pin="S"/>
+<pinref part="S3" gate="G$1" pin="S"/>
 </segment>
 <segment>
@@
 <wire x1="20.32" y1="17.78" x2="20.32" y2="15.24" width="0.1524" layer="91"/>
 <junction x="20.32" y="15.24"/>
+</segment>
+<segment>
+<pinref part="J1" gate="G$1" pin="C"/>
+<pinref part="GND_1" gate="1" pin="GND"/>
+<wire x1="22.86" y1="43.18" x2="27.94" y2="43.18" width="0.1524" layer="91"/>
 </segment>
 </net>
@@
 <junction x="20.32" y="27.94"/>
 </segment>
+<segment>
+<pinref part="J1" gate="G$1" pin="A"/>
+<pinref part="P+2" gate="1" pin="+5V"/>
+<wire x1="22.86" y1="48.26" x2="27.94" y2="48.26" width="0.1524" layer="91"/>
+</segment>
 </net>
 <net name="DOT" class="0">
@@
 </segment>
 <segment>
-<pinref part="S1" gate="G$1" pin="2"/>
-<wire x1="177.8" y1="22.86" x2="182.88" y2="22.86" width="0.1524" layer="91"/>
-<label x="182.88" y="22.86" size="1.27" layer="95" xref="yes"/>
+<pinref part="S1" gate="G$1" pin="P"/>
+<wire x1="180.34" y1="20.32" x2="175.26" y2="20.32" width="0.1524" layer="91"/>
+<label x="175.26" y="20.32" size="1.27" layer="95" rot="R180" xref="yes"/>
 </segment>
 </net>
@@
 </segment>
 <segment>
-<pinref part="S2" gate="G$1" pin="2"/>
-<wire x1="167.64" y1="15.24" x2="172.72" y2="15.24" width="0.1524" layer="91"/>
-<label x="172.72" y="15.24" size="1.27" layer="95" xref="yes"/>
+<pinref part="S2" gate="G$1" pin="P"/>
+<wire x1="172.72" y1="12.7" x2="167.64" y2="12.7" width="0.1524" layer="91"/>
+<label x="167.64" y="12.7" size="1.27" layer="95" rot="R180" xref="yes"/>
 </segment>
 </net>
@@
 </segment>
 <segment>
-<pinref part="S3" gate="G$1" pin="2"/>
-<wire x1="157.48" y1="7.62" x2="165.1" y2="7.62" width="0.1524" layer="91"/>
-<label x="165.1" y="7.62" size="1.27" layer="95" xref="yes"/>
-</segment>
-</net>
+<pinref part="S3" gate="G$1" pin="P"/>
+<wire x1="167.64" y1="5.08" x2="162.56" y2="5.08" width="0.1524" layer="91"/>
+<label x="162.56" y="5.08" size="1.27" layer="95" rot="R180" xref="yes"/>
+</segment>
+</net>

Commit message: corrected pcb
Connections:
- net GND: now also J1.B
Changed lines of the file:
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@@
 <pinref part="J1" gate="G$1" pin="C"/>
 <pinref part="GND_1" gate="1" pin="GND"/>
-<wire x1="22.86" y1="43.18" x2="27.94" y2="43.18" width="0.1524" layer="91"/>
+<wire x1="22.86" y1="43.18" x2="25.4" y2="43.18" width="0.1524" layer="91"/>
+<pinref part="J1" gate="G$1" pin="B"/>
+<wire x1="25.4" y1="43.18" x2="27.94" y2="43.18" width="0.1524" layer="91"/>
+<wire x1="22.86" y1="45.72" x2="25.4" y2="45.72" width="0.1524" layer="91"/>
+<wire x1="25.4" y1="45.72" x2="25.4" y2="43.18" width="0.1524" layer="91"/>
+<junction x="25.4" y="43.18"/>
 </segment>
 </net>
