File: eagle/HighVBoard_02.brd (EAGLE design)
At the start: 113 x 48.3 mm, 22 parts, among them IC2 K155D1, IC3 K155D1, IC4 K155D1, IC5 K155D1, Q1 VN2224, T1 INS-3

Commit message: pcb updates
Parts:
- removed JACK: (no value), pinhead:1X02/90
- removed Q1: VN2224, Nixie:TO92
- added U$2: NIXIE-PSU, Nixie:NIXIE-PSU
- U$1: value NIXIE-PSU -> SSN1N45BTA; device Nixie:NIXIE-PSU -> Nixie:TO92
- moved U$1 22.1 mm to (56.5, 17.8), turned to 180 degrees
- moved R1 0.64 mm to (18.4, 35.6)
- moved R2 0.64 mm to (38.7, 35.6)
- moved R3 0.64 mm to (74.3, 35.6)
- moved R4 0.64 mm to (94.6, 35.6)
- moved TP_170V 0.64 mm to (69.2, 42.5)
- moved TP_GND 0.64 mm to (43.8, 40.0)
- moved HOUR1 0.64 mm to (15.9, 24.8)
- moved HOUR2 0.64 mm to (38.7, 24.8)
- moved MINUTE1 0.64 mm to (74.3, 24.8)
- moved MINUTE2 0.64 mm to (97.2, 24.8)
- moved T1 0.64 mm to (56.5, 24.8)
- moved IC2 0.63 mm to (21.0, 10.8)
- moved IC3 0.63 mm to (43.8, 10.8)
- moved IC4 0.63 mm to (69.2, 10.8)
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Connections:
- net +170V: now also U$2.5; no longer U$1.5
- net +5V: now also U$2.1; no longer JACK.1, U$1.1
- net DOT: now also U$1.3; no longer Q1.2
- net GND: now also U$1.1, U$2.2, U$2.4; no longer JACK.2, Q1.1, U$1.2, U$1.4
- net N$1: now also U$1.2; no longer Q1.3
Routing:
- net GND: track 152.5 -> 136.3 mm
- net HOUR1_C: track 22.1 -> 28.6 mm
- net +170V: track 103.5 -> 97.9 mm
- net +5V: track 162.8 -> 158.3 mm
- net N$46: track 21.8 -> 25.6 mm
- net N$1: track 5.71 -> 9.42 mm
- net DOT: track 13.5 -> 15.6 mm
- net N$29: track 23.0 -> 24.6 mm
- net N$23: track 12.9 -> 14.5 mm
- net N$12: track 12.9 -> 14.5 mm
- net N$49: track 8.67 -> 9.94 mm
- net N$51: track 27.6 -> 28.9 mm
- net N$45: track 9.69 -> 11.0 mm
- net N$39: track 19.2 -> 20.5 mm
- net N$35: track 19.7 -> 21.0 mm
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Other:
- board size 113 x 48.3 mm -> 113 x 52.1 mm

Commit message: corrected pcb
Parts:
- removed HOUR1, HOUR2, MINUTE1, MINUTE2: IN-8, Nixie:IN-8
- added T2, T3, T4, T5: IN-8, Nixie:IN-8
- moved POWER 1.27 mm to (38.7, 45.1)
- moved U$2 1.27 mm to (50.2, 40.0)
- moved DATA 1.27 mm to (56.5, 3.94)
- moved IC2 1.27 mm to (21.0, 12.1)
- moved IC3 1.27 mm to (43.8, 12.1)
- moved IC4 1.27 mm to (69.2, 12.1)
- moved IC5 1.27 mm to (92.1, 12.1)
- moved R5 1.27 mm to (61.6, 25.4)
- moved T1 1.27 mm to (56.5, 26.0)
- moved U$1 1.27 mm to (56.5, 19.1)
- moved R1 1.27 mm to (18.4, 36.8)
- moved R2 1.27 mm to (38.7, 36.8)
- moved R3 1.27 mm to (74.3, 36.8)
- moved R4 1.27 mm to (94.6, 36.8)
- moved TP_170V 1.27 mm to (69.2, 43.8)
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Connections:
- net N$10: now also T2.1; no longer HOUR1.1
- net N$11: now also T2.2; no longer HOUR1.2
- net N$12: now also T2.3; no longer HOUR1.3
- net N$13: now also T2.4; no longer HOUR1.4
- net N$14: now also T2.5; no longer HOUR1.5
- net N$15: now also T2.6; no longer HOUR1.6
- net N$16: now also T2.7; no longer HOUR1.7
- net N$17: now also T2.8; no longer HOUR1.8
- net N$18: now also T2.9; no longer HOUR1.9
- net N$19: now also T2.A; no longer HOUR1.A
- net N$20: now also T3.10; no longer HOUR2.10
- net N$21: now also T3.1; no longer HOUR2.1
- net N$22: now also T3.2; no longer HOUR2.2
- net N$23: now also T3.3; no longer HOUR2.3
- net N$24: now also T3.4; no longer HOUR2.4
- net N$25: now also T3.5; no longer HOUR2.5
- net N$26: now also T3.6; no longer HOUR2.6
- net N$27: now also T3.7; no longer HOUR2.7
- net N$28: now also T3.8; no longer HOUR2.8
- net N$29: now also T3.9; no longer HOUR2.9
- net N$30: now also T3.A; no longer HOUR2.A
- net N$31: now also T4.10; no longer MINUTE1.10
- net N$32: now also T4.1; no longer MINUTE1.1
- net N$33: now also T4.2; no longer MINUTE1.2
- net N$34: now also T4.3; no longer MINUTE1.3
- net N$35: now also T4.4; no longer MINUTE1.4
- net N$36: now also T4.5; no longer MINUTE1.5
- net N$37: now also T4.6; no longer MINUTE1.6
- net N$38: now also T4.7; no longer MINUTE1.7
- net N$39: now also T4.8; no longer MINUTE1.8
- net N$40: now also T4.9; no longer MINUTE1.9
- net N$41: now also T4.A; no longer MINUTE1.A
- net N$42: now also T5.10; no longer MINUTE2.10
- net N$43: now also T5.1; no longer MINUTE2.1
- net N$44: now also T5.2; no longer MINUTE2.2
- net N$45: now also T5.3; no longer MINUTE2.3
- net N$46: now also T5.4; no longer MINUTE2.4
- net N$47: now also T5.5; no longer MINUTE2.5
- net N$48: now also T5.6; no longer MINUTE2.6
- net N$49: now also T5.7; no longer MINUTE2.7
- net N$50: now also T5.8; no longer MINUTE2.8
- net N$51: now also T5.9; no longer MINUTE2.9
- net N$52: now also T5.A; no longer MINUTE2.A
- net N$7: now also T2.10; no longer HOUR1.10
Routing:
- net N$46: track 25.6 -> 7.92 mm
- net N$28: track 16.3 -> 33.7 mm
- net N$17: track 16.2 -> 33.0 mm
- net N$35: track 21.0 -> 8.19 mm
- net N$42: track 16.6 -> 29.2 mm
- net N$34: track 11.0 -> 22.3 mm
- net N$45: track 11.0 -> 22.1 mm
- net N$16: track 22.1 -> 11.0 mm
- net N$27: track 22.1 -> 11.2 mm
- net N$18: track 25.2 -> 35.8 mm
- net N$31: track 18.9 -> 29.5 mm
- net N$23: track 14.5 -> 24.8 mm
- net N$33: track 21.8 -> 31.8 mm
- net N$44: track 22.3 -> 31.9 mm
- net N$12: track 14.5 -> 23.9 mm
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Other:
- outline, holes or cut-outs redrawn

Commit message: updated pcb and partslist
Parts:
- R1, R2, R3, R4: value 8.2k -> 10.2k
- moved U$1 0.23 mm to (56.5, 19.3), turned to 0 degrees
Connections:
- net DOT: now also U$1.1; no longer U$1.3
- net GND: now also U$1.3; no longer U$1.1
Routing:
- net N$1: track 9.42 -> 5.38 mm
- net GND: track 136.3 -> 136.9 mm
Other:
- board text added: "R1.2.1"
- board text removed: "R1.2"
Changed lines of the file:
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@@
 <text x="95.25" y="33.02" size="1.778" layer="25" font="vector" align="center">IN-8</text>
 <text x="95.885" y="1.905" size="1.778" layer="25" font="vector" align="center">ZENO GRIES</text>
-<text x="12.7" y="1.905" size="1.778" layer="25" font="vector" align="center">R1.2</text>
+<text x="13.97" y="1.905" size="1.778" layer="25" font="vector" align="center">R1.2.1</text>
 <wire x1="88.265" y1="38.735" x2="94.615" y2="48.895" width="0.1524" layer="21"/>
 <wire x1="94.615" y1="48.895" x2="100.965" y2="38.735" width="0.1524" layer="21"/>
@@
 <attribute name="VALUE" x="92.075" y="12.065" size="1.778" layer="25" font="vector" align="center"/>
 </element>
-<element name="R1" library="resistor" library_urn="urn:adsk.eagle:library:348" package="0207/10" package3d_urn="urn:adsk.eagle:package:23491/1" value="8.2k" x="18.415" y="36.83" smashed="yes">
+<element name="R1" library="resistor" library_urn="urn:adsk.eagle:library:348" package="0207/10" package3d_urn="urn:adsk.eagle:package:23491/1" value="10.2k" x="18.415" y="36.83" smashed="yes">
 <attribute name="VALUE" x="18.415" y="36.83" size="1.27" layer="25" font="vector" align="center"/>
 </element>
-<element name="R2" library="resistor" library_urn="urn:adsk.eagle:library:348" package="0207/10" package3d_urn="urn:adsk.eagle:package:23491/1" value="8.2k" x="38.735" y="36.83" smashed="yes">
+<element name="R2" library="resistor" library_urn="urn:adsk.eagle:library:348" package="0207/10" package3d_urn="urn:adsk.eagle:package:23491/1" value="10.2k" x="38.735" y="36.83" smashed="yes">
 <attribute name="VALUE" x="38.735" y="36.83" size="1.27" layer="25" font="vector" align="center"/>
 </element>
-<element name="R3" library="resistor" library_urn="urn:adsk.eagle:library:348" package="0207/10" package3d_urn="urn:adsk.eagle:package:23491/1" value="8.2k" x="74.295" y="36.83" smashed="yes">
+<element name="R3" library="resistor" library_urn="urn:adsk.eagle:library:348" package="0207/10" package3d_urn="urn:adsk.eagle:package:23491/1" value="10.2k" x="74.295" y="36.83" smashed="yes">
 <attribute name="VALUE" x="74.295" y="36.83" size="1.27" layer="25" font="vector" align="center"/>
 </element>
-<element name="R4" library="resistor" library_urn="urn:adsk.eagle:library:348" package="0207/10" package3d_urn="urn:adsk.eagle:package:23491/1" value="8.2k" x="94.615" y="36.83" smashed="yes">
+<element name="R4" library="resistor" library_urn="urn:adsk.eagle:library:348" package="0207/10" package3d_urn="urn:adsk.eagle:package:23491/1" value="10.2k" x="94.615" y="36.83" smashed="yes">
 <attribute name="VALUE" x="94.615" y="36.83" size="1.27" layer="25" font="vector" align="center"/>
 </element>
@@
 <attribute name="VALUE" x="35.56" y="47.625" size="1.27" layer="27" rot="R270"/>
 </element>
-<element name="U$1" library="Nixie" package="TO92" value="SSN1N45BTA" x="56.515" y="19.05" smashed="yes" rot="R180">
-<attribute name="VALUE" x="54.864" y="21.59" size="1.27" layer="27" font="vector" rot="R180" align="center"/>
-</element>
 <element name="U$2" library="Nixie" package="NIXIE-PSU" value="NIXIE-PSU" x="50.165" y="40.005" smashed="yes" rot="R270"/>
 <element name="T2" library="Nixie" package="IN-8" value="IN-8" x="17.78" y="26.035" smashed="yes">
-<attribute name="NAME" x="17.78" y="36.035" size="1.27" layer="21" align="bottom-center"/>
 <attribute name="VALUE" x="17.78" y="16.035" size="1.27" layer="21" align="top-center"/>
 </element>
 <element name="T3" library="Nixie" package="IN-8" value="IN-8" x="40.005" y="26.035" smashed="yes">
-<attribute name="NAME" x="40.005" y="36.035" size="1.27" layer="21" align="bottom-center"/>
 <attribute name="VALUE" x="40.005" y="16.035" size="1.27" layer="21" align="top-center"/>
 </element>
 <element name="T4" library="Nixie" package="IN-8" value="IN-8" x="73.025" y="26.035" smashed="yes">
-<attribute name="NAME" x="73.025" y="36.035" size="1.27" layer="21" align="bottom-center"/>
 <attribute name="VALUE" x="73.025" y="16.035" size="1.27" layer="21" align="top-center"/>
 </element>
 <element name="T5" library="Nixie" package="IN-8" value="IN-8" x="95.25" y="26.035" smashed="yes">
-<attribute name="NAME" x="95.25" y="36.035" size="1.27" layer="21" align="bottom-center"/>
 <attribute name="VALUE" x="95.25" y="16.035" size="1.27" layer="21" align="top-center"/>
+</element>
+<element name="U$1" library="Nixie" package="TO92" value="SSN1N45BTA" x="56.515" y="19.2786" smashed="yes">
+<attribute name="NAME" x="58.928" y="20.9296" size="1.27" layer="25" ratio="10"/>
+<attribute name="VALUE" x="59.436" y="18.0086" size="1.27" layer="27" ratio="10"/>
 </element>
 </elements>
@@
 <wire x1="45.085" y1="15.875" x2="45.085" y2="12.0396" width="0.4064" layer="16"/>
 <wire x1="70.485" y1="15.875" x2="70.485" y2="12.0396" width="0.4064" layer="16"/>
-<contactref element="U$1" pad="1"/>
-<wire x1="57.785" y1="19.05" x2="53.975" y2="22.86" width="0.4064" layer="1"/>
-<wire x1="57.785" y1="19.05" x2="57.785" y2="12.0396" width="0.4064" layer="16"/>
 <contactref element="U$2" pad="2"/>
 <contactref element="U$2" pad="4"/>
 <wire x1="43.815" y1="41.275" x2="45.085" y2="42.545" width="0.4064" layer="16"/>
 <wire x1="45.085" y1="42.545" x2="50.165" y2="42.545" width="0.4064" layer="16"/>
-<wire x1="53.975" y1="22.86" x2="53.975" y2="35.56" width="0.4064" layer="1"/>
+<wire x1="53.975" y1="35.56" x2="53.975" y2="22.1334875" width="0.4064" layer="1"/>
 <wire x1="53.975" y1="35.56" x2="52.07" y2="37.465" width="0.4064" layer="1"/>
 <wire x1="52.07" y1="37.465" x2="50.165" y2="37.465" width="0.4064" layer="1"/>
 <wire x1="50.165" y1="37.465" x2="47.625" y2="37.465" width="0.4064" layer="16"/>
 <wire x1="47.625" y1="37.465" x2="43.815" y2="41.275" width="0.4064" layer="16"/>
+<contactref element="U$1" pad="3"/>
+<wire x1="57.785" y1="19.2786" x2="57.785" y2="12.0396" width="0.4064" layer="16"/>
+<wire x1="57.785" y1="19.2786" x2="56.8298875" y2="19.2786" width="0.4064" layer="1"/>
+<wire x1="56.8298875" y1="19.2786" x2="53.975" y2="22.1334875" width="0.4064" layer="1"/>
 </signal>
 <signal name="N$7" class="3">
@@
 <signal name="N$1">
 <contactref element="T1" pad="C"/>
-<contactref element="U$1" pad="2"/>
 <wire x1="56.515" y1="22.987" x2="55.245" y2="24.257" width="0.2032" layer="16"/>
 <wire x1="55.245" y1="26.035" x2="55.245" y2="24.257" width="0.2032" layer="16"/>
-<wire x1="56.515" y1="22.987" x2="56.515" y2="17.145" width="0.2032" layer="16"/>
+<contactref element="U$1" pad="2"/>
+<wire x1="56.515" y1="21.1836" x2="56.515" y2="22.987" width="0.2032" layer="16"/>
 </signal>
 <signal name="DOT">
 <contactref element="DATA" pad="9"/>
-<contactref element="U$1" pad="3"/>
-<wire x1="55.245" y1="19.05" x2="55.245" y2="17.0434" width="0.2032" layer="1"/>
-<wire x1="55.245" y1="17.0434" x2="56.515" y2="15.7734" width="0.2032" layer="1"/>
-<wire x1="56.515" y1="15.7734" x2="56.515" y2="3.937" width="0.2032" layer="1"/>
+<contactref element="U$1" pad="1"/>
+<wire x1="56.515" y1="18.0086" x2="55.245" y2="19.2786" width="0.2032" layer="1"/>
+<wire x1="56.515" y1="3.937" x2="56.515" y2="18.0086" width="0.2032" layer="1"/>
 </signal>
 <signal name="+170V" class="3">
