File: eagle/HighVBoard_02.sch (EAGLE design)
At the start: 22 parts, among them IC2 K155D1, IC3 K155D1, IC4 K155D1, IC5 K155D1, Q1 VN2224, T1 INS-3

Commit message: pcb updates
Parts:
- removed JACK: (no value), pinhead:PINHD-1X2/90
- removed Q1: VN2224, Nixie:VN2224
- added U$2: NIXIE-PSU, Nixie:NIXIE-PSU
- U$1: value NIXIE-PSU -> SSN1N45BTA; device Nixie:NIXIE-PSU -> Nixie:SSN1N45BTA
Connections:
- net +170V: now also U$2.OUT; no longer U$1.OUT
- net +5V: now also U$2.IN; no longer JACK.1, U$1.IN
- net DOT: now also U$1.G; no longer Q1.G
- net GND: now also U$1.S, U$2.GND; no longer JACK.2, Q1.S, U$1.GND
- net N$1: now also U$1.D; no longer Q1.D
Changed lines of the file:
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@@
 <part name="TP_170V" library="testpad" library_urn="urn:adsk.eagle:library:385" deviceset="TP" device="PAD1-13" package3d_urn="urn:adsk.eagle:package:27946/1"/>
 <part name="P+2" library="supply1" library_urn="urn:adsk.eagle:library:371" deviceset="+5V" device=""/>
-<part name="P+4" library="supply1" library_urn="urn:adsk.eagle:library:371" deviceset="+5V" device=""/>
-<part name="GND_4" library="supply1" library_urn="urn:adsk.eagle:library:371" deviceset="GND" device=""/>
 <part name="P+5" library="supply1" library_urn="urn:adsk.eagle:library:371" deviceset="+5V" device=""/>
 <part name="GND_5" library="supply1" library_urn="urn:adsk.eagle:library:371" deviceset="GND" device=""/>
@@
 <part name="P+6" library="supply1" library_urn="urn:adsk.eagle:library:371" deviceset="+5V" device=""/>
 <part name="GND_6" library="supply1" library_urn="urn:adsk.eagle:library:371" deviceset="GND" device=""/>
-<part name="Q1" library="Nixie" deviceset="VN2224" device=""/>
 <part name="HOUR1" library="Nixie" deviceset="IN-8" device=""/>
 <part name="HOUR2" library="Nixie" deviceset="IN-8" device=""/>
 <part name="MINUTE1" library="Nixie" deviceset="IN-8" device=""/>
 <part name="MINUTE2" library="Nixie" deviceset="IN-8" device=""/>
-<part name="U$1" library="Nixie" deviceset="NIXIE-PSU" device=""/>
 <part name="T1" library="Nixie" deviceset="INS-3" device=""/>
 <part name="POWER" library="pinhead" library_urn="urn:adsk.eagle:library:325" deviceset="PINHD-1X2" device="" package3d_urn="urn:adsk.eagle:package:22435/2"/>
-<part name="JACK" library="pinhead" library_urn="urn:adsk.eagle:library:325" deviceset="PINHD-1X2" device="/90" package3d_urn="urn:adsk.eagle:package:22437/2"/>
+<part name="U$1" library="Nixie" deviceset="SSN1N45BTA" device=""/>
+<part name="U$2" library="Nixie" deviceset="NIXIE-PSU" device=""/>
 </parts>
 <sheets>
@@
 <attribute name="VALUE" x="134.62" y="25.4" size="1.778" layer="96" rot="R180"/>
 </instance>
-<instance part="P+4" gate="1" x="127" y="154.94" smashed="yes" rot="R90">
-<attribute name="VALUE" x="127" y="157.48" size="1.778" layer="96" rot="R180"/>
-</instance>
-<instance part="GND_4" gate="1" x="127" y="152.4" smashed="yes" rot="R270">
-<attribute name="VALUE" x="124.46" y="154.94" size="1.778" layer="96" rot="R270"/>
-</instance>
 <instance part="P+5" gate="1" x="182.88" y="134.62" smashed="yes">
 <attribute name="VALUE" x="180.34" y="129.54" size="1.778" layer="96" rot="R90"/>
@@
 <attribute name="VALUE" x="142.24" y="114.3" size="1.778" layer="96"/>
 </instance>
-<instance part="Q1" gate="G$1" x="337.82" y="63.5" smashed="yes">
-<attribute name="VALUE" x="326.39" y="63.5" size="1.778" layer="96"/>
-<attribute name="NAME" x="326.39" y="66.04" size="1.778" layer="95"/>
-</instance>
 <instance part="HOUR1" gate="G$1" x="162.56" y="86.36" smashed="yes" rot="R90">
 <attribute name="NAME" x="142.24" y="85.0646" size="1.778" layer="95" rot="R90" align="bottom-center"/>
@@
 <attribute name="VALUE" x="317.5" y="85.09" size="1.6764" layer="96" rot="R90" align="top-center"/>
 </instance>
-<instance part="U$1" gate="G$1" x="144.78" y="134.62" smashed="yes"/>
 <instance part="T1" gate="G$1" x="340.36" y="83.82" smashed="yes">
 <attribute name="NAME" x="334.772" y="78.74" size="1.778" layer="95" rot="R90"/>
@@
 <attribute name="VALUE" x="186.69" y="121.92" size="1.778" layer="96"/>
 </instance>
-<instance part="JACK" gate="G$1" x="167.64" y="152.4" smashed="yes">
-<attribute name="NAME" x="161.29" y="158.115" size="1.778" layer="95"/>
-<attribute name="VALUE" x="161.29" y="147.32" size="1.778" layer="96"/>
-</instance>
+<instance part="U$1" gate="G$1" x="337.82" y="63.5" smashed="yes">
+<attribute name="VALUE" x="326.39" y="63.5" size="1.778" layer="96"/>
+<attribute name="NAME" x="326.39" y="66.04" size="1.778" layer="95"/>
+</instance>
+<instance part="U$2" gate="G$1" x="144.78" y="134.62" smashed="yes"/>
 </instances>
 <busses>
@@
 <junction x="137.16" y="10.16"/>
 <wire x1="340.36" y1="58.42" x2="340.36" y2="10.16" width="0.1524" layer="91"/>
-<pinref part="Q1" gate="G$1" pin="S"/>
-</segment>
-<segment>
-<pinref part="GND_4" gate="1" pin="GND"/>
-<wire x1="165.1" y1="152.4" x2="129.54" y2="152.4" width="0.1524" layer="91"/>
-<pinref part="JACK" gate="G$1" pin="2"/>
+<pinref part="U$1" gate="G$1" pin="S"/>
 </segment>
 <segment>
@@
 </segment>
 <segment>
-<pinref part="U$1" gate="G$1" pin="GND"/>
-<wire x1="144.78" y1="124.46" x2="144.78" y2="119.38" width="0.1524" layer="91"/>
+<pinref part="U$2" gate="G$1" pin="GND"/>
 <pinref part="GND_6" gate="1" pin="GND"/>
+<wire x1="144.78" y1="119.38" x2="144.78" y2="124.46" width="0.1524" layer="91"/>
 </segment>
 </net>
@@
 </segment>
 <segment>
-<pinref part="P+4" gate="1" pin="+5V"/>
-<wire x1="165.1" y1="154.94" x2="129.54" y2="154.94" width="0.1524" layer="91"/>
-<pinref part="JACK" gate="G$1" pin="1"/>
-</segment>
-<segment>
 <pinref part="P+5" gate="1" pin="+5V"/>
 <wire x1="182.88" y1="132.08" x2="182.88" y2="129.54" width="0.1524" layer="91"/>
@@
 <wire x1="134.62" y1="134.62" x2="129.54" y2="134.62" width="0.1524" layer="91"/>
 <pinref part="P+6" gate="1" pin="+5V"/>
-<pinref part="U$1" gate="G$1" pin="IN"/>
+<pinref part="U$2" gate="G$1" pin="IN"/>
 </segment>
 </net>
@@
 <segment>
 <wire x1="340.36" y1="68.58" x2="340.36" y2="76.2" width="0.1524" layer="91"/>
-<pinref part="Q1" gate="G$1" pin="D"/>
 <pinref part="T1" gate="G$1" pin="C"/>
+<pinref part="U$1" gate="G$1" pin="D"/>
 </segment>
 </net>
@@
 <wire x1="332.74" y1="60.96" x2="327.66" y2="60.96" width="0.1524" layer="91"/>
 <label x="327.66" y="60.96" size="1.27" layer="95" rot="R180" xref="yes"/>
-<pinref part="Q1" gate="G$1" pin="G"/>
+<pinref part="U$1" gate="G$1" pin="G"/>
 </segment>
 <segment>
@@
 <wire x1="154.94" y1="134.62" x2="160.02" y2="134.62" width="0.1524" layer="91"/>
 <label x="160.02" y="134.62" size="1.778" layer="95" xref="yes"/>
-<pinref part="U$1" gate="G$1" pin="OUT"/>
-</segment>
-<segment>
+<pinref part="U$2" gate="G$1" pin="OUT"/>
+</segment>
+<segment>

Commit message: corrected pcb
Parts:
- renumbered HOUR1 to T2, HOUR2 to T3, MINUTE1 to T4, MINUTE2 to T5

Commit message: updated pcb and partslist
Parts:
- R1, R2, R3, R4: value 8.2k -> 10.2k
Changed lines of the file:
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@@
 <part name="GND_1" library="supply1" library_urn="urn:adsk.eagle:library:371" deviceset="GND" device=""/>
 <part name="IC2" library="Nixie" deviceset="K155D1" device=""/>
-<part name="R1" library="resistor" library_urn="urn:adsk.eagle:library:348" deviceset="R-EU_" device="0207/10" package3d_urn="urn:adsk.eagle:package:23491/1" value="8.2k"/>
+<part name="R1" library="resistor" library_urn="urn:adsk.eagle:library:348" deviceset="R-EU_" device="0207/10" package3d_urn="urn:adsk.eagle:package:23491/1" value="10.2k"/>
 <part name="IC3" library="Nixie" deviceset="K155D1" device=""/>
-<part name="R2" library="resistor" library_urn="urn:adsk.eagle:library:348" deviceset="R-EU_" device="0207/10" package3d_urn="urn:adsk.eagle:package:23491/1" value="8.2k"/>
+<part name="R2" library="resistor" library_urn="urn:adsk.eagle:library:348" deviceset="R-EU_" device="0207/10" package3d_urn="urn:adsk.eagle:package:23491/1" value="10.2k"/>
 <part name="IC4" library="Nixie" deviceset="K155D1" device=""/>
-<part name="R3" library="resistor" library_urn="urn:adsk.eagle:library:348" deviceset="R-EU_" device="0207/10" package3d_urn="urn:adsk.eagle:package:23491/1" value="8.2k"/>
+<part name="R3" library="resistor" library_urn="urn:adsk.eagle:library:348" deviceset="R-EU_" device="0207/10" package3d_urn="urn:adsk.eagle:package:23491/1" value="10.2k"/>
 <part name="IC5" library="Nixie" deviceset="K155D1" device=""/>
-<part name="R4" library="resistor" library_urn="urn:adsk.eagle:library:348" deviceset="R-EU_" device="0207/10" package3d_urn="urn:adsk.eagle:package:23491/1" value="8.2k"/>
+<part name="R4" library="resistor" library_urn="urn:adsk.eagle:library:348" deviceset="R-EU_" device="0207/10" package3d_urn="urn:adsk.eagle:package:23491/1" value="10.2k"/>
 <part name="R5" library="resistor" library_urn="urn:adsk.eagle:library:348" deviceset="R-EU_" device="0207/10" package3d_urn="urn:adsk.eagle:package:23491/1" value="130k"/>
 <part name="TP_GND" library="testpad" library_urn="urn:adsk.eagle:library:385" deviceset="TP" device="PAD1-13" package3d_urn="urn:adsk.eagle:package:27946/1"/>
@@
 <part name="T1" library="Nixie" deviceset="INS-3" device=""/>
 <part name="POWER" library="pinhead" library_urn="urn:adsk.eagle:library:325" deviceset="PINHD-1X2" device="" package3d_urn="urn:adsk.eagle:package:22435/2"/>
-<part name="U$1" library="Nixie" deviceset="SSN1N45BTA" device=""/>
 <part name="U$2" library="Nixie" deviceset="NIXIE-PSU" device=""/>
 <part name="T2" library="Nixie" deviceset="IN-8" device=""/>
@@
 <part name="T4" library="Nixie" deviceset="IN-8" device=""/>
 <part name="T5" library="Nixie" deviceset="IN-8" device=""/>
+<part name="U$1" library="Nixie" deviceset="SSN1N45BTA" device=""/>
 </parts>
 <sheets>
@@
 <attribute name="VALUE" x="186.69" y="121.92" size="1.778" layer="96"/>
 </instance>
-<instance part="U$1" gate="G$1" x="337.82" y="63.5" smashed="yes">
-<attribute name="VALUE" x="326.39" y="63.5" size="1.778" layer="96"/>
-<attribute name="NAME" x="326.39" y="66.04" size="1.778" layer="95"/>
-</instance>
 <instance part="U$2" gate="G$1" x="144.78" y="134.62" smashed="yes"/>
 <instance part="T2" gate="G$1" x="162.56" y="86.36" smashed="yes" rot="R90">
@@
 <attribute name="VALUE" x="317.5" y="85.09" size="1.6764" layer="96" rot="R90" align="top-center"/>
 </instance>
+<instance part="U$1" gate="G$1" x="337.82" y="63.5" smashed="yes">
+<attribute name="VALUE" x="326.39" y="63.5" size="1.778" layer="96"/>
+<attribute name="NAME" x="326.39" y="66.04" size="1.778" layer="95"/>
+</instance>
 </instances>
