File: eagle/HighVBoard_1.4.brd (EAGLE design)
At the start: 113 x 52.1 mm, 21 parts, among them IC2 K155D1, IC3 K155D1, IC4 K155D1, IC5 K155D1, T1 INS-3, T2 IN-8, T3 IN-8, T4 IN-8, T5 IN-8

Commit message: new boards
Parts:
- added ENABLE: (no value), pinhead:1X01
- moved R2 1.27 mm to (40.0, 36.8)
- moved R3 1.27 mm to (73.0, 36.8)
- moved R4 0.64 mm to (95.2, 36.8)
- moved R1 0.63 mm to (17.8, 36.8)
- moved U$2 0.63 mm to (49.5, 40.0)
Connections:
- new net N$2: ENABLE.1, U$2.3
Routing:
- net N$2: track 0.00 -> 20.8 mm
- net N$30: track 11.5 -> 10.2 mm
- net MINUTE1_A: track 10.3 -> 9.12 mm
- net HOUR2_A: track 10.1 -> 8.97 mm
- net HOUR2_D: track 10.1 -> 9.05 mm
- net HOUR2_C: track 7.56 -> 6.51 mm
- net N$41: track 9.25 -> 10.2 mm
- net +170V: track 99.6 -> 100.5 mm
- net HOUR2_B: track 7.37 -> 6.51 mm
- net MINUTE1_C: track 12.4 -> 11.6 mm
- net MINUTE1_B: track 12.5 -> 11.7 mm
- net MINUTE1_D: track 9.78 -> 9.08 mm
- net +5V: track 158.5 -> 157.9 mm
- net N$52: track 10.9 -> 10.2 mm
- net N$19: track 9.59 -> 10.2 mm
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Other:
- board text added: "R1.4"
- board text removed: "R1.3"
