File: eagle/HighVBoard_1.4.sch (EAGLE design)
At the start: 21 parts, among them IC2 K155D1, IC3 K155D1, IC4 K155D1, IC5 K155D1, T1 INS-3, T2 IN-8, T3 IN-8, T4 IN-8, T5 IN-8

Commit message: new boards
Parts:
- added ENABLE: (no value), pinhead:PINHD-1X1
Connections:
- new net N$2: ENABLE.1, U$2.EN
Changed lines of the file:
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@@
 <?xml version="1.0" encoding="utf-8"?>
 <!DOCTYPE eagle SYSTEM "eagle.dtd">
-<eagle version="9.2.2">
+<eagle version="9.6.2">
 <drawing>
 <settings>
@@
 <part name="T5" library="Nixie" deviceset="IN-8" device=""/>
 <part name="U$1" library="Nixie" deviceset="SSN1N45BTA" device=""/>
+<part name="ENABLE" library="pinhead" library_urn="urn:adsk.eagle:library:325" deviceset="PINHD-1X1" device="" package3d_urn="urn:adsk.eagle:package:22485/2"/>
 </parts>
 <sheets>
@@
 <attribute name="VALUE" x="326.39" y="63.5" size="1.778" layer="96"/>
 <attribute name="NAME" x="326.39" y="66.04" size="1.778" layer="95"/>
+</instance>
+<instance part="ENABLE" gate="G$1" x="144.78" y="157.48" smashed="yes" rot="R90">
+<attribute name="NAME" x="141.605" y="151.13" size="1.778" layer="95" rot="R90"/>
+<attribute name="VALUE" x="149.86" y="151.13" size="1.778" layer="96" rot="R90"/>
 </instance>
 </instances>
@@
 </segment>
 </net>
+<net name="N$2" class="0">
+<segment>
+<pinref part="U$2" gate="G$1" pin="EN"/>
+<pinref part="ENABLE" gate="G$1" pin="1"/>
+<wire x1="144.78" y1="144.78" x2="144.78" y2="154.94" width="0.1524" layer="91"/>
+</segment>
+</net>
