File: eagle/LowVBoard_1.4.brd (EAGLE design)
At the start: 113 x 52.1 mm, 29 parts, among them IC1 ATMEGA328P-PU, IC2 MCP7940M, IC3 SN74HC595, IC4 SN74HC595, J1 CONNJACKR/APCB5.5X2.1MM, Q1 16MHz, Q2 32.768kHz

Commit message: new boards
Parts:
- added DEBUG: (no value), pinhead:1X11/90
- added ENABLE, ENABLE_DEBUG: (no value), pinhead:1X01
- added ENABLE_JUMPER: (no value), pinhead:1X02
- added POWER_D: (no value), pinhead:1X02/90
- moved C2 33.8 mm to (45.1, 8.64), turned to 270 degrees
- moved C1 29.1 mm to (40.8, 8.51), turned to 0 degrees
- moved R1 17.7 mm to (11.4, 20.4), turned to 90 degrees
- moved IC1 13.7 mm to (31.1, 16.5)
- moved IC4 11.4 mm to (61.0, 21.6), turned to 90 degrees
- moved R2 10.6 mm to (14.6, 28.6), turned to 90 degrees
- moved R3 9.67 mm to (17.1, 27.9), turned to 90 degrees
- moved R4 9.09 mm to (19.7, 27.3), turned to 90 degrees
- moved D1 8.28 mm to (91.4, 29.8), turned to 0 degrees
- moved C3 5.12 mm to (33.0, 6.99), turned to 270 degrees
- moved C4 5.12 mm to (17.8, 6.99), turned to 270 degrees
- moved Q1 5.08 mm to (25.4, 6.99)
- moved C6 2.01 mm to (85.1, 14.6)
- moved Q2 2.01 mm to (88.9, 15.9)
- moved C5 2.01 mm to (92.7, 14.6)
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Connections:
- removed net N$57: IC1.28, IC2.6, R2.1
- removed net N$58: IC1.27, IC2.5, R3.1
- removed net N$59: IC1.26, IC2.7, R4.1
- new net ENABLE: ENABLE.1, ENABLE_JUMPER.1
- new net ENABLE_ATMEGA: ENABLE_DEBUG.1, ENABLE_JUMPER.2, IC1.15
- new net MFP: DEBUG.8, IC1.26, IC2.7, R4.1
- new net SCL: DEBUG.10, IC1.28, IC2.6, R2.1
- new net SDA: DEBUG.9, IC1.27, IC2.5, R3.1
- net +5V: now also POWER_D.2
- net CLOCK: now also DEBUG.2
- net DATA: now also DEBUG.1
- net DOT: now also DEBUG.4
- net GND: now also DEBUG.11, POWER_D.1
- net LATCH: now also DEBUG.3
- net SWITCH1: now also DEBUG.5
- net SWITCH2: now also DEBUG.6
- net SWITCH3: now also DEBUG.7
Routing:
- net N$57: track 106.7 -> 0.00 mm
- net N$58: track 100.3 -> 0.00 mm
- net SCL: track 0.00 -> 99.4 mm, vias 0 -> 1
- net SDA: track 0.00 -> 97.3 mm, vias 0 -> 1
- net N$59: track 89.7 -> 0.00 mm
- net MFP: track 0.00 -> 80.2 mm, vias 0 -> 1
- net +5V: track 169.3 -> 225.0 mm, vias 1 -> 2
- net GND: track 380.5 -> 329.0 mm, vias 1 -> 3
- net MINUTE1_B: track 65.6 -> 21.6 mm, vias 1 -> 0
- net MINUTE1_A: track 14.6 -> 56.5 mm
- net ENABLE_ATMEGA: track 0.00 -> 33.7 mm, vias 0 -> 1
- net HOUR1_A: track 14.6 -> 41.4 mm
- net MINUTE2_C: track 29.6 -> 53.2 mm
- net N$56: track 28.6 -> 5.95 mm
- net MINUTE2_B: track 26.7 -> 47.1 mm
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Other:
- board text added: "17/A3 MFP"
- board text added: "2 DATA"
- board text added: "3 CLOCK"
- board text added: "4 LATCH"
- board text added: "5 DOT"
- board text added: "5V"
- board text added: "6 SWITCH1"
- board text added: "7 SWITCH2"
- board text added: "8 SWITCH3"
- board text added: "9 ENABLE"
- board text added: "GND"
- board text added: "R1.4"
- board text added: "SCL"
- board text added: "SDA"
- board text removed: "R1.3"
