File: eagle/LowVBoard_1.4.sch (EAGLE design)
At the start: 29 parts, among them IC1 ATMEGA328P-PU, IC2 MCP7940M, IC3 SN74HC595, IC4 SN74HC595, J1 CONNJACKR/APCB5.5X2.1MM, Q1 16MHz, Q2 32.768kHz

Commit message: new boards
Parts:
- added DEBUG: (no value), pinhead:PINHD-1X11/90
- added ENABLE, ENABLE_DEBUG: (no value), pinhead:PINHD-1X1
- added ENABLE_JUMPER: (no value), pinhead:PINHD-1X2
- added POWER_D: (no value), pinhead:PINHD-1X2/90
Connections:
- removed net N$57: IC1.19/A5/SCL, IC2.SCL, R2.1
- removed net N$58: IC1.18/A4/SDA, IC2.SDA, R3.1
- removed net N$59: IC1.17/A3, IC2.MFP, R4.1
- new net ENABLE: ENABLE.1, ENABLE_JUMPER.1
- new net ENABLE_ATMEGA: ENABLE_DEBUG.1, ENABLE_JUMPER.2, IC1.~9
- new net MFP: DEBUG.8, IC1.17/A3, IC2.MFP, R4.1
- new net SCL: DEBUG.10, IC1.19/A5/SCL, IC2.SCL, R2.1
- new net SDA: DEBUG.9, IC1.18/A4/SDA, IC2.SDA, R3.1
- net +5V: now also POWER_D.2
- net CLOCK: now also DEBUG.2
- net DATA: now also DEBUG.1
- net DOT: now also DEBUG.4
- net GND: now also DEBUG.11, POWER_D.1
- net LATCH: now also DEBUG.3
- net SWITCH1: now also DEBUG.5
- net SWITCH2: now also DEBUG.6
- net SWITCH3: now also DEBUG.7
