File: kicad/Nixie IN-8.kicad_pcb (KiCad board)
At the start: 2 copper layers, 116.8 x 91.4 mm, 47 parts, among them J1 Conn_01x03_Pin, J2 Conn_01x02_Pin, J3 Conn_01x03_Pin, J4 Conn_01x04_Pin, J5 Conn_01x04_Pin, J6 Barrel_Jack_Switch, Q1 MPSA42, SW1 SW_SPST, SW2 SW_SPST, SW3 SW_SPST, U1 K155ID1, U2 K155ID1, U3 K155ID1, U4 K155ID1, U5 MCP7940N, U6 74HC595, U7 74HC595, Y1 32.768kHz

Commit message: setup board
Parts:
- removed the REF** at (189.2, 47.0)
- removed U7: 74HC595, Package_SO:SOIC-16_3.9x9.9mm_P1.27mm
- removed mouse-bite-2.54mm-slot1, mouse-bite-2.54mm-slot2, mouse-bite-2.54mm-slot3: VAL**, Panelization:mouse-bite-2.54mm-slot
- added C5: 0.1µF, Capacitor_THT:C_Disc_D3.0mm_W1.6mm_P2.50mm, F.Cu at (163.8, 85.1)
- added C6: 6pF, Capacitor_SMD:C_1206_3216Metric_Pad1.33x1.80mm_HandSolder, B.Cu at (170.7, 125.8)
- added C7: 6pF, Capacitor_SMD:C_1206_3216Metric_Pad1.33x1.80mm_HandSolder, B.Cu at (177.7, 125.8)
- added Q10: MPSA42, Package_TO_SOT_THT:TO-92_Inline_Wide, F.Cu at (87.6, 57.8)
- added Q11: MPSA42, Package_TO_SOT_THT:TO-92_Inline_Wide, F.Cu at (109.9, 57.8)
- added Q12: MPSA42, Package_TO_SOT_THT:TO-92_Inline_Wide, F.Cu at (142.9, 57.8)
- added Q13: MPSA42, Package_TO_SOT_THT:TO-92_Inline_Wide, F.Cu at (165.1, 57.8)
- added Q14: MPSA42, Package_TO_SOT_THT:TO-92_Inline_Wide, F.Cu at (88.3, 70.5)
- added Q15: MPSA42, Package_TO_SOT_THT:TO-92_Inline_Wide, F.Cu at (110.5, 70.5)
- added Q16: MPSA42, Package_TO_SOT_THT:TO-92_Inline_Wide, F.Cu at (143.5, 70.5)
- added Q17: MPSA42, Package_TO_SOT_THT:TO-92_Inline_Wide, F.Cu at (165.7, 70.5)
- added Q18: MPSA42, Package_TO_SOT_THT:TO-92_Inline_Wide, F.Cu at (86.4, 78.1)
- added Q19: MPSA42, Package_TO_SOT_THT:TO-92_Inline_Wide, F.Cu at (108.6, 78.1)
- added Q2: MPSA42, Package_TO_SOT_THT:TO-92_Inline_Wide, F.Cu at (127.0, 53.6)
- added Q20: MPSA42, Package_TO_SOT_THT:TO-92_Inline_Wide, F.Cu at (141.6, 78.1)
- added Q21: MPSA42, Package_TO_SOT_THT:TO-92_Inline_Wide, F.Cu at (163.8, 78.1)
- added Q22: MPSA42, Package_TO_SOT_THT:TO-92_Inline_Wide, F.Cu at (91.4, 78.1)
- added Q23: MPSA42, Package_TO_SOT_THT:TO-92_Inline_Wide, F.Cu at (113.7, 78.1)
- added Q24: MPSA42, Package_TO_SOT_THT:TO-92_Inline_Wide, F.Cu at (146.7, 78.1)
- added Q25: MPSA42, Package_TO_SOT_THT:TO-92_Inline_Wide, F.Cu at (168.9, 78.1)
- added Q26: MPSA42, Package_TO_SOT_THT:TO-92_Inline_Wide, F.Cu at (96.5, 78.1)
- added Q27: MPSA42, Package_TO_SOT_THT:TO-92_Inline_Wide, F.Cu at (118.7, 78.1)
- added Q28: MPSA42, Package_TO_SOT_THT:TO-92_Inline_Wide, F.Cu at (151.8, 78.1)
- added Q29: MPSA42, Package_TO_SOT_THT:TO-92_Inline_Wide, F.Cu at (174.0, 78.1)
- added Q3: MPSA42, Package_TO_SOT_THT:TO-92_Inline_Wide, F.Cu at (160.0, 53.6)
- added Q30: MPSA42, Package_TO_SOT_THT:TO-92_Inline_Wide, F.Cu at (101.6, 78.1)
- added Q31: MPSA42, Package_TO_SOT_THT:TO-92_Inline_Wide, F.Cu at (123.8, 78.1)
- added Q32: MPSA42, Package_TO_SOT_THT:TO-92_Inline_Wide, F.Cu at (156.8, 78.1)
- added Q33: MPSA42, Package_TO_SOT_THT:TO-92_Inline_Wide, F.Cu at (179.1, 78.1)
- added Q34: MPSA42, Package_TO_SOT_THT:TO-92_Inline_Wide, F.Cu at (105.1, 70.5)
- added Q35: MPSA42, Package_TO_SOT_THT:TO-92_Inline_Wide, F.Cu at (127.4, 70.5)
- added Q36: MPSA42, Package_TO_SOT_THT:TO-92_Inline_Wide, F.Cu at (160.4, 70.5)
- added Q37: MPSA42, Package_TO_SOT_THT:TO-92_Inline_Wide, F.Cu at (182.6, 70.5)
- added Q38: MPSA42, Package_TO_SOT_THT:TO-92_Inline_Wide, F.Cu at (104.4, 57.8)
- added Q39: MPSA42, Package_TO_SOT_THT:TO-92_Inline_Wide, F.Cu at (126.6, 57.8)
- added Q4: MPSA42, Package_TO_SOT_THT:TO-92_Inline_Wide, F.Cu at (182.2, 53.6)
- added Q40: MPSA42, Package_TO_SOT_THT:TO-92_Inline_Wide, F.Cu at (159.7, 57.8)
- added Q41: MPSA42, Package_TO_SOT_THT:TO-92_Inline_Wide, F.Cu at (181.9, 57.8)
- added Q5: MPSA42, Package_TO_SOT_THT:TO-92_Inline_Wide, F.Cu at (133.3, 74.9)
- added Q6: MPSA42, Package_TO_SOT_THT:TO-92_Inline_Wide, F.Cu at (89.5, 54.2)
- added Q7: MPSA42, Package_TO_SOT_THT:TO-92_Inline_Wide, F.Cu at (111.8, 54.2)
- added Q8: MPSA42, Package_TO_SOT_THT:TO-92_Inline_Wide, F.Cu at (144.8, 54.2)
- added Q9: MPSA42, Package_TO_SOT_THT:TO-92_Inline_Wide, F.Cu at (167.0, 54.2)
- added R10: 22k, Resistor_THT:R_Axial_DIN0204_L3.6mm_D1.6mm_P5.08mm_Vertical, F.Cu at (129.6, 77.5)
- added R11: 10k, Resistor_SMD:R_1206_3216Metric_Pad1.30x1.75mm_HandSolder, B.Cu at (142.2, 100.7)
- added R12: 10k, Resistor_SMD:R_1206_3216Metric_Pad1.30x1.75mm_HandSolder, B.Cu at (139.7, 100.7)
- added R13: 10k, Resistor_SMD:R_1206_3216Metric_Pad1.30x1.75mm_HandSolder, B.Cu at (144.8, 100.7)
- added REF**: MountingHole_3.2mm_M3_Pad, MountingHole:MountingHole_3.2mm_M3_Pad, F.Cu at (189.2, 47.0)
- added mouse-bite-2.54mm-slot: VAL**, Panelization:mouse-bite-2.54mm-slot, F.Cu at (120.7, 90.2)
- added mouse-bite-2.54mm-slot: VAL**, Panelization:mouse-bite-2.54mm-slot, F.Cu at (154.3, 90.2)
- added mouse-bite-2.54mm-slot: VAL**, Panelization:mouse-bite-2.54mm-slot, F.Cu at (188.0, 90.2)
- C3, C4: value 6pF -> 0.1µF; footprint Capacitor_SMD:C_1206_3216Metric_Pad1.33x1.80mm_HandSolder -> Capacitor_THT:C_Disc_D3.0mm_W1.6mm_P2.50mm; moved to F.Cu
- J2: value Conn_01x02_Pin -> Conn_01x04_Pin; footprint Connector_PinHeader_2.54mm:PinHeader_1x02_P2.54mm_Horizontal -> Connector_PinHeader_2.54mm:PinHeader_1x04_P2.54mm_Vertical; moved to F.Cu
- J5: value Conn_01x04_Pin -> Conn_01x02_Pin; footprint Connector_PinHeader_2.54mm:PinHeader_1x04_P2.54mm_Vertical -> Connector_PinHeader_2.54mm:PinHeader_1x02_P2.54mm_Horizontal; moved to B.Cu
- R4: value 10k -> 12k; footprint Resistor_SMD:R_1206_3216Metric_Pad1.30x1.75mm_HandSolder -> Resistor_THT:R_Axial_DIN0207_L6.3mm_D2.5mm_P10.16mm_Horizontal; moved to F.Cu
- R5: value 10k -> 200k; footprint Resistor_SMD:R_1206_3216Metric_Pad1.30x1.75mm_HandSolder -> Resistor_THT:R_Axial_DIN0207_L6.3mm_D2.5mm_P10.16mm_Horizontal; moved to F.Cu
- R6: value 10k -> 22k; footprint Resistor_SMD:R_1206_3216Metric_Pad1.30x1.75mm_HandSolder -> Resistor_THT:R_Axial_DIN0204_L3.6mm_D1.6mm_P5.08mm_Vertical; moved to F.Cu
- R7: value 12k -> 22k; footprint Resistor_THT:R_Axial_DIN0207_L6.3mm_D2.5mm_P10.16mm_Horizontal -> Resistor_THT:R_Axial_DIN0204_L3.6mm_D1.6mm_P5.08mm_Vertical
- R9: value 200k -> 22k; footprint Resistor_THT:R_Axial_DIN0207_L6.3mm_D2.5mm_P10.16mm_Horizontal -> Resistor_THT:R_Axial_DIN0204_L3.6mm_D1.6mm_P5.08mm_Vertical
- TP2: value 5V -> 12V
- TP3: value GND -> 5V
- TP4: value 12V -> GND
- U1, U2, U3, U4: value K155ID1 -> 74HC595; footprint Package_DIP:DIP-16_W7.62mm_Socket -> Package_SO:SOIC-16_3.9x9.9mm_P1.27mm
- U5: value MCP7940N -> 74HC595; footprint Package_SO:SOIC-8_3.9x4.9mm_P1.27mm -> Package_SO:SOIC-16_3.9x9.9mm_P1.27mm; moved to F.Cu
- U6: value 74HC595 -> MCP7940N-xP; footprint Package_SO:SOIC-16_3.9x9.9mm_P1.27mm -> Package_SO:SOIC-8_3.9x4.9mm_P1.27mm; moved to B.Cu
- moved J1 90.8 mm to (132.1, 47.0), turned to -90 degrees
- moved J3 90.8 mm to (163.8, 132.1), turned to 90 degrees
- moved U6 74.1 mm to (172.0, 118.6), turned to 90 degrees
- moved R6 69.0 mm to (82.5, 73.1)
- moved R4 59.4 mm to (174.6, 50.2)
- moved C3 58.3 mm to (125.1, 85.1), turned to 90 degrees
- moved TP2 57.3 mm to (80.0, 52.1)
- moved C2 50.7 mm to (111.8, 85.1)
- moved R5 47.5 mm to (133.3, 52.7)
- moved R9 46.9 mm to (182.2, 73.1), turned to -90 degrees
- moved R7 45.7 mm to (127.0, 73.0), turned to -90 degrees
- moved TP3 45.2 mm to (136.5, 47.0)
- moved C4 38.6 mm to (150.4, 85.1), turned to 90 degrees
- moved J5 33.1 mm to (124.5, 102.8), turned to 90 degrees
- moved Q1 32.8 mm to (104.8, 53.6)
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Connections:
- C3 pad 1: Net-(U5-X1) -> /5V_1
- C3 pad 2: GND2 -> GND1
- C4 pad 1: Net-(U5-X2) -> /5V_1
- C4 pad 2: GND2 -> GND1
- J1 pad 1: /5V_2 -> /5V_1
- J1 pad 2: GND2 -> GND1
- J1 pad 3: /12V_2 -> /12V_1
- J2 pad 1: Net-(A1-+5V) -> /DATA
- J2 pad 2: /5V_2 -> /CLOCK
- J3 pad 1: /5V_1 -> /5V_2
- J3 pad 2: GND1 -> GND2
- J3 pad 3: /12V_1 -> /12V_2
- J4 pad 1: /DATA -> /MCU_DATA
- J4 pad 2: /CLOCK -> /MCU_CLOCK
- J4 pad 3: /LATCH -> /MCU_LATCH
- J4 pad 4: /DOT -> /MCU_DOT
- J5 pad 1: /MCU_DATA -> Net-(A1-+5V)
- J5 pad 2: /MCU_CLOCK -> /5V_2
- Q1 pad 1: GND1 -> /HOUR1.0
- R4 pad 1: /5V_2 -> /180V
- R4 pad 2: /SCL -> Net-(R4-Pad2)
- R5 pad 1: /5V_2 -> /180V
- R5 pad 2: /SDA -> Net-(R5-Pad2)
- R6 pad 1: /5V_2 -> Net-(Q1-B)
- R6 pad 2: /MFP -> /5V_1
- R7 pad 1: /180V -> Net-(Q11-B)
- R7 pad 2: Net-(R7-Pad2) -> /5V_1
- R8 pad 1: Net-(Q1-B) -> Net-(Q12-B)
- R8 pad 2: /DOT -> /5V_1
- R9 pad 1: /180V -> Net-(Q13-B)
- R9 pad 2: Net-(R9-Pad2) -> /5V_1
- SW1 pad 1: /SWITCH.1 -> /SWITCH.3
- SW3 pad 1: /SWITCH.3 -> /SWITCH.1
- TP2 pad 1: /5V_1 -> /12V_1
- TP3 pad 1: GND1 -> /5V_1
- TP4 pad 1: /12V_1 -> GND1
- U1 pad 1: Net-(U1-8) -> /HOUR1.1
- U1 pad 10: Net-(U1-7) -> unconnected-(U1-~{SRCLR}-Pad10)
- U1 pad 11: Net-(U1-6) -> /CLOCK
- U1 pad 12: GND1 -> /LATCH
- U1 pad 13: Net-(U1-4) -> GND1
- U1 pad 14: Net-(U1-5) -> /DATA
- U1 pad 15: Net-(U1-1) -> /HOUR1.0
- U1 pad 16: Net-(U1-0) -> /5V_1
- U1 pad 2: Net-(U1-9) -> /HOUR1.2
- U1 pad 3: /HOUR1.A -> /HOUR1.3
- U1 pad 4: /HOUR1.D -> /HOUR1.4
- U1 pad 5: /5V_1 -> /HOUR1.5
- U1 pad 6: /HOUR1.B -> /HOUR1.6
- U1 pad 7: /HOUR1.C -> /HOUR1.7
- U1 pad 8: Net-(U1-2) -> GND1
- U1 pad 9: Net-(U1-3) -> Net-(U1-QH')
- U2 pad 1: Net-(U2-8) -> /HOUR1.9
- U2 pad 10: Net-(U2-7) -> unconnected-(U2-~{SRCLR}-Pad10)
- U2 pad 11: Net-(U2-6) -> /CLOCK
- U2 pad 12: GND1 -> /LATCH
- U2 pad 13: Net-(U2-4) -> GND1
- U2 pad 14: Net-(U2-5) -> Net-(U1-QH')
- U2 pad 15: Net-(U2-1) -> /HOUR1.8
- U2 pad 16: Net-(U2-0) -> /5V_1
- U2 pad 2: Net-(U2-9) -> /HOUR2.0
- U2 pad 3: /HOUR2.A -> /HOUR2.1
- U2 pad 4: /HOUR2.D -> /HOUR2.2
- U2 pad 5: /5V_1 -> /HOUR2.3
- U2 pad 6: /HOUR2.B -> /HOUR2.4
- U2 pad 7: /HOUR2.C -> /HOUR2.5
- U2 pad 8: Net-(U2-2) -> GND1
- U2 pad 9: Net-(U2-3) -> Net-(U2-QH')
- U3 pad 1: Net-(U3-8) -> /HOUR2.7
- U3 pad 10: Net-(U3-7) -> unconnected-(U3-~{SRCLR}-Pad10)
- U3 pad 11: Net-(U3-6) -> /CLOCK
- U3 pad 12: GND1 -> /LATCH
- U3 pad 13: Net-(U3-4) -> GND1
- U3 pad 14: Net-(U3-5) -> Net-(U2-QH')
- U3 pad 15: Net-(U3-1) -> /HOUR2.6
- U3 pad 16: Net-(U3-0) -> /5V_1
- U3 pad 2: Net-(U3-9) -> /HOUR2.8
- U3 pad 3: /MINUTE1.A -> /HOUR2.9
- U3 pad 4: /MINUTE1.D -> /MINUTE1.0
- U3 pad 5: /5V_1 -> /MINUTE1.1
- U3 pad 6: /MINUTE1.B -> /MINUTE1.2
- U3 pad 7: /MINUTE1.C -> /MINUTE1.3
- U3 pad 8: Net-(U3-2) -> GND1
- U3 pad 9: Net-(U3-3) -> Net-(U3-QH')
- U4 pad 1: Net-(U4-8) -> /MINUTE1.5
- U4 pad 10: Net-(U4-7) -> unconnected-(U4-~{SRCLR}-Pad10)
- U4 pad 11: Net-(U4-6) -> /CLOCK
- U4 pad 12: GND1 -> /LATCH
- U4 pad 13: Net-(U4-4) -> GND1
- U4 pad 14: Net-(U4-5) -> Net-(U3-QH')
- U4 pad 15: Net-(U4-1) -> /MINUTE1.4
- U4 pad 16: Net-(U4-0) -> /5V_1
- U4 pad 2: Net-(U4-9) -> /MINUTE1.6
- U4 pad 3: /MINUTE2.A -> /MINUTE1.7
- U4 pad 4: /MINUTE2.D -> /MINUTE1.8
- U4 pad 5: /5V_1 -> /MINUTE1.9
- U4 pad 6: /MINUTE2.B -> /MINUTE2.0
- U4 pad 7: /MINUTE2.C -> /MINUTE2.1
- U4 pad 8: Net-(U4-2) -> GND1
- U4 pad 9: Net-(U4-3) -> Net-(U4-QH')
- U5 pad 1: Net-(U5-X1) -> /MINUTE2.3
- U5 pad 2: Net-(U5-X2) -> /MINUTE2.4
- U5 pad 3: Net-(BT1-+) -> /MINUTE2.5
- U5 pad 4: GND2 -> /MINUTE2.6
- U5 pad 5: /SDA -> /MINUTE2.7
- U5 pad 6: /SCL -> /MINUTE2.8
- U5 pad 7: /MFP -> /MINUTE2.9
- U5 pad 8: /5V_2 -> GND1
- U6 pad 1: /HOUR1.B -> Net-(U6-X1)
- U6 pad 2: /HOUR1.C -> Net-(U6-X2)
- U6 pad 3: /HOUR1.D -> Net-(BT1-+)
- U6 pad 4: /HOUR2.A -> GND2
- U6 pad 5: /HOUR2.B -> /SDA
- U6 pad 6: /HOUR2.C -> /SCL
- U6 pad 7: /HOUR2.D -> /MFP
- U6 pad 8: GND1 -> /5V_2
- V1 pad 1: Net-(U1-1) -> Net-(Q6-C)
- V1 pad 10: Net-(U1-0) -> Net-(Q1-C)
- V1 pad 2: Net-(U1-2) -> Net-(Q10-C)
- V1 pad 3: Net-(U1-3) -> Net-(Q14-C)
- V1 pad 4: Net-(U1-4) -> Net-(Q18-C)
- V1 pad 5: Net-(U1-5) -> Net-(Q22-C)
- V1 pad 6: Net-(U1-6) -> Net-(Q26-C)
- V1 pad 7: Net-(U1-7) -> Net-(Q30-C)
- V1 pad 8: Net-(U1-8) -> Net-(Q34-C)
- V1 pad 9: Net-(U1-9) -> Net-(Q38-C)
- V2 pad 1: Net-(U2-1) -> Net-(Q7-C)
- V2 pad 10: Net-(U2-0) -> Net-(Q2-C)
- V2 pad 2: Net-(U2-2) -> Net-(Q11-C)
- V2 pad 3: Net-(U2-3) -> Net-(Q15-C)
- V2 pad 4: Net-(U2-4) -> Net-(Q19-C)
- V2 pad 5: Net-(U2-5) -> Net-(Q23-C)
- V2 pad 6: Net-(U2-6) -> Net-(Q27-C)
- V2 pad 7: Net-(U2-7) -> Net-(Q31-C)
- V2 pad 8: Net-(U2-8) -> Net-(Q35-C)
- V2 pad 9: Net-(U2-9) -> Net-(Q39-C)
- V3 pad 1: Net-(U3-1) -> Net-(Q8-C)
- V3 pad 10: Net-(U3-0) -> Net-(Q3-C)
- V3 pad 2: Net-(U3-2) -> Net-(Q12-C)
- V3 pad 3: Net-(U3-3) -> Net-(Q16-C)
- V3 pad 4: Net-(U3-4) -> Net-(Q20-C)
- V3 pad 5: Net-(U3-5) -> Net-(Q24-C)
- V3 pad 6: Net-(U3-6) -> Net-(Q28-C)
- V3 pad 7: Net-(U3-7) -> Net-(Q32-C)
- V3 pad 8: Net-(U3-8) -> Net-(Q36-C)
- V3 pad 9: Net-(U3-9) -> Net-(Q40-C)
- V4 pad 1: Net-(U4-1) -> Net-(Q9-C)
- V4 pad 10: Net-(U4-0) -> Net-(Q4-C)
- V4 pad 2: Net-(U4-2) -> Net-(Q13-C)
- V4 pad 3: Net-(U4-3) -> Net-(Q17-C)
- V4 pad 4: Net-(U4-4) -> Net-(Q21-C)
- V4 pad 5: Net-(U4-5) -> Net-(Q25-C)
- V4 pad 6: Net-(U4-6) -> Net-(Q29-C)
- V4 pad 7: Net-(U4-7) -> Net-(Q33-C)
- V4 pad 8: Net-(U4-8) -> Net-(Q37-C)
- V4 pad 9: Net-(U4-9) -> Net-(Q41-C)
- V4 pad A: Net-(R7-Pad2) -> Net-(R4-Pad2)
- V5 pad A: Net-(R9-Pad2) -> Net-(R5-Pad2)
- V5 pad C: Net-(Q1-C) -> Net-(Q5-C)
- Y1 pad 1: Net-(U5-X1) -> Net-(U6-X1)
- Y1 pad 2: Net-(U5-X2) -> Net-(U6-X2)
Routing:
- net Net-(Q11-B): track 0.00 -> 75.1 mm
- net Net-(Q13-B): track 0.00 -> 75.1 mm
- net Net-(Q12-B): track 0.00 -> 75.1 mm
- net Net-(Q1-B): track 7.67 -> 75.1 mm
- net Net-(U6-QH'): track 64.8 -> 0.00 mm, vias 2 -> 0
- net /HOUR1.1: track 0.00 -> 53.4 mm
- net /MINUTE2.0: track 0.00 -> 50.4 mm
- net /MINUTE2.9: track 0.00 -> 44.9 mm
- net /MINUTE1.0: track 0.00 -> 43.9 mm
- net /HOUR1.2: track 0.00 -> 41.8 mm
- net /HOUR1.0: track 0.00 -> 40.1 mm
- net /HOUR1.9: track 0.00 -> 38.6 mm
- net /MINUTE1.2: track 0.00 -> 36.8 mm
- net /HOUR1.3: track 0.00 -> 36.7 mm
- net /MINUTE2.2: track 0.00 -> 36.3 mm
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
Commit message: finished routing
Parts:
- removed A1: ARDUINO NANO EVERY, Nixie:Arduino_Nano_SMT
- removed mouse-bite-2.54mm-slot (x3): VAL**, Panelization:mouse-bite-2.54mm-slot
- added D1: D, Diode_SMD:D_SMA_Handsoldering, B.Cu at (161.3, 127.0)
- added J7: Conn_01x04_Pin, Connector_PinHeader_2.54mm:PinHeader_1x04_P2.54mm_Vertical, F.Cu at (156.2, 97.2)
- added J8: Conn_01x02_Pin, Connector_PinHeader_2.54mm:PinHeader_1x02_P2.54mm_Vertical, F.Cu at (117.5, 95.9)
- added J9: Barrel_Jack_Switch, Connector_BarrelJack:BarrelJack_Wuerth_6941xx301002, B.Cu at (186.7, 120.6)
- added U7: Pico, MCU_RaspberryPi_and_Boards:RPi_Pico_SMD, B.Cu at (128.9, 113.1)
- J3: value Conn_01x03_Pin -> Conn_01x04_Pin; footprint Connector_PinHeader_2.54mm:PinHeader_1x03_P2.54mm_Vertical -> Connector_PinHeader_2.54mm:PinHeader_1x04_P2.54mm_Vertical
- J4: value Conn_01x04_Pin -> Conn_01x02_Pin; footprint Connector_PinHeader_2.54mm:PinHeader_1x04_P2.54mm_Vertical -> Connector_PinHeader_2.54mm:PinHeader_1x02_P2.54mm_Vertical
- J5: value Conn_01x02_Pin -> Conn_01x03_Pin; footprint Connector_PinHeader_2.54mm:PinHeader_1x02_P2.54mm_Horizontal -> Connector_PinHeader_2.54mm:PinHeader_1x03_P2.54mm_Vertical
- J6: value Barrel_Jack_Switch -> Conn_01x04_Pin; footprint Connector_BarrelJack:BarrelJack_Wuerth_6941xx301002 -> Connector_PinHeader_2.54mm:PinHeader_1x04_P2.54mm_Vertical; moved to F.Cu
- R10, R6, R7, R8, R9: value 22k -> 13.5k
- moved J3 55.7 mm to (139.7, 81.9)
- moved J5 49.1 mm to (163.8, 132.1), turned to -90 degrees
- moved J6 40.8 mm to (156.2, 93.3), turned to -90 degrees
- moved R11 28.0 mm to (163.8, 118.5)
- moved R12 28.0 mm to (161.3, 118.5)
- moved R13 28.0 mm to (166.4, 118.5)
- moved J4 24.4 mm to (178.4, 83.2), turned to 0 degrees
- moved C4 1.02 mm to (150.5, 86.1)
- moved C5 1.02 mm to (163.8, 86.1)
- moved C2 0.91 mm to (111.8, 86.0)
- moved C3 0.90 mm to (125.0, 86.0)
- moved U1 0.45 mm to (104.8, 83.6)
- moved U2 0.45 mm to (118.1, 83.6)
- moved U3 0.45 mm to (131.4, 83.6)
- moved U4 0.45 mm to (156.8, 83.6)
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Connections:
- C1 pad 1: /5V_1 -> /3.3V_1
- C2 pad 1: /5V_1 -> /3.3V_1
- C3 pad 1: /5V_1 -> /3.3V_1
- C4 pad 1: /5V_1 -> /3.3V_1
- C5 pad 1: /5V_1 -> /3.3V_1
- J3 pad 1: /5V_2 -> /HOUR1_EN
- J3 pad 2: GND2 -> /HOUR2_EN
- J3 pad 3: /12V_2 -> /MINUTE1_EN
- J4 pad 1: /MCU_DATA -> /3.3V_1
- J4 pad 2: /MCU_CLOCK -> /OE
- J5 pad 1: Net-(A1-+5V) -> /5V_2
- J5 pad 2: /5V_2 -> GND2
- J6 pad 1: /12V_2 -> /MCU_DATA
- J6 pad 2: GND2 -> /MCU_CLOCK
- J6 pad 3: GND2 -> /MCU_LATCH
- R11 pad 1: /5V_2 -> /3.3V_2
- R12 pad 1: /5V_2 -> /3.3V_2
- R13 pad 1: /5V_2 -> /3.3V_2
- R6 pad 2: /5V_1 -> /HOUR1_EN
- R7 pad 2: /5V_1 -> /HOUR2_EN
- R8 pad 2: /5V_1 -> /MINUTE1_EN
- R9 pad 2: /5V_1 -> /MINUTE2_EN
- U1 pad 13: GND1 -> /OE
- U1 pad 16: /5V_1 -> /3.3V_1
- U2 pad 13: GND1 -> /OE
- U2 pad 16: /5V_1 -> /3.3V_1
- U3 pad 13: GND1 -> /OE
- U3 pad 16: /5V_1 -> /3.3V_1
- U4 pad 13: GND1 -> /OE
- U4 pad 16: /5V_1 -> /3.3V_1
- U5 pad 13: GND1 -> /OE
- U5 pad 16: /5V_1 -> /3.3V_1
- U6 pad 8: /5V_2 -> /3.3V_2
Routing:
- net /5V_2: track 109.7 -> 5.10 mm, vias 2 -> 0
- net /5V_1: track 209.8 -> 108.3 mm, vias 5 -> 0
- net /3.3V_1: track 0.00 -> 94.0 mm, vias 0 -> 5
- net /3.3V_2: track 0.00 -> 88.6 mm
- net /OE: track 0.00 -> 80.5 mm, vias 0 -> 5
- net /HOUR1_EN: track 0.00 -> 61.0 mm
- net Net-(D1-K): track 0.00 -> 60.4 mm
- net /MINUTE2_EN: track 0.00 -> 42.6 mm
- net /MCU_OE: track 0.00 -> 42.4 mm
- net GND2: track 0.00 -> 37.9 mm, vias 0 -> 3
- net GND1: track 283.2 -> 314.5 mm, vias 10 -> 4
- net Net-(A1-+5V): track 26.8 -> 0.00 mm, vias 1 -> 0
- net /HOUR2_EN: track 0.00 -> 18.4 mm
- net /MCU_MINUTE2_EN: track 0.00 -> 16.0 mm
- net /MCU_MINUTE1_EN: track 0.00 -> 16.0 mm
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Other:
- outline, holes or cut-outs redrawn

Commit message: finished routing
Parts:
- removed J6, J7: Conn_01x04_Pin, Connector_PinHeader_2.54mm:PinHeader_1x04_P2.54mm_Vertical
- removed J8: Conn_01x02_Pin, Connector_PinHeader_2.54mm:PinHeader_1x02_P2.54mm_Vertical
- removed J9: Barrel_Jack_Switch, Connector_BarrelJack:BarrelJack_Wuerth_6941xx301002
- removed Q10, Q11, Q12, Q13, Q14, Q15, Q16, Q17, Q18, Q19, Q2, Q20, Q21, Q22, Q23, Q24, Q25, Q26, Q27, Q28, Q29, Q3, Q30, Q31, Q32, Q33, Q34, Q35, Q36, Q37, Q38, Q39, Q4, Q40, Q41, Q5, Q6, Q7, Q8, Q9: MPSA42, Package_TO_SOT_THT:TO-92_Inline_Wide
- removed R10: 13.5k, Resistor_THT:R_Axial_DIN0204_L3.6mm_D1.6mm_P5.08mm_Vertical
- removed R11, R12, R13: 10k, Resistor_SMD:R_1206_3216Metric_Pad1.30x1.75mm_HandSolder
- added C8: 6pF, Capacitor_SMD:C_1206_3216Metric_Pad1.33x1.80mm_HandSolder, B.Cu at (124.8, 104.8)
- added C9: 0.1µF, Capacitor_SMD:C_1206_3216Metric_Pad1.33x1.80mm_HandSolder, B.Cu at (131.7, 104.8)
- added REF**: MountingHole_3.2mm_M3, MountingHole:MountingHole_3.2mm_M3, F.Cu at (186.7, 82.5)
- added REF**: MountingHole_3.2mm_M3, MountingHole:MountingHole_3.2mm_M3, F.Cu at (186.7, 127.0)
- added REF**: MountingHole_3.2mm_M3, MountingHole:MountingHole_3.2mm_M3, F.Cu at (186.7, 49.5)
- added REF**: MountingHole_3.2mm_M3, MountingHole:MountingHole_3.2mm_M3, F.Cu at (101.6, 82.5)
- added REF**: MountingHole_3.2mm_M3, MountingHole:MountingHole_3.2mm_M3, F.Cu at (186.7, 94.0)
- added U8: MCP7940N-xP, Package_SO:SOIC-8_3.9x4.9mm_P1.27mm, B.Cu at (132.0, 99.7)
- added mouse-bite-2.54mm-slot: VAL**, Panelization:mouse-bite-2.54mm-slot, F.Cu at (186.1, 88.3)
- added mouse-bite-2.54mm-slot: VAL**, Panelization:mouse-bite-2.54mm-slot, F.Cu at (118.7, 88.3)
- added mouse-bite-2.54mm-slot: VAL**, Panelization:mouse-bite-2.54mm-slot, F.Cu at (152.4, 88.3)
- C6: value 6pF -> 0.1µF
- J1: value Conn_01x03_Pin -> Conn_01x05_Pin; footprint Connector_PinHeader_2.54mm:PinHeader_1x03_P2.54mm_Vertical -> Connector_PinHeader_2.54mm:PinHeader_1x05_P2.54mm_Vertical
- J2, J3: value Conn_01x04_Pin -> Conn_01x03_Pin; footprint Connector_PinHeader_2.54mm:PinHeader_1x04_P2.54mm_Vertical -> Connector_PinHeader_2.54mm:PinHeader_1x03_P2.54mm_Vertical
- J4: value Conn_01x02_Pin -> Conn_01x05_Pin; footprint Connector_PinHeader_2.54mm:PinHeader_1x02_P2.54mm_Vertical -> Connector_PinHeader_2.54mm:PinHeader_1x05_P2.54mm_Vertical
- J5: value Conn_01x03_Pin -> Barrel_Jack_Switch; footprint Connector_PinHeader_2.54mm:PinHeader_1x03_P2.54mm_Vertical -> Connector_BarrelJack:BarrelJack_Wuerth_6941xx301002
- R1, R2, R3, R4: value 12k -> 8.66k
- R5: value 200k -> 162k
- R6: footprint Resistor_THT:R_Axial_DIN0204_L3.6mm_D1.6mm_P5.08mm_Vertical -> Resistor_THT:R_Axial_DIN0204_L3.6mm_D1.6mm_P5.08mm_Horizontal
- R7, R8, R9: value 13.5k -> 10k; footprint Resistor_THT:R_Axial_DIN0204_L3.6mm_D1.6mm_P5.08mm_Vertical -> Resistor_SMD:R_1206_3216Metric_Pad1.30x1.75mm_HandSolder; moved to B.Cu
- TP1: value 180V -> 170V
- U1, U2, U3, U4, U5: value 74HC595 -> TPIC6B595; footprint Package_SO:SOIC-16_3.9x9.9mm_P1.27mm -> Package_SO:SOIC-20W_7.5x12.8mm_P1.27mm
- U6: value MCP7940N-xP -> SN74AHCT125; footprint Package_SO:SOIC-8_3.9x4.9mm_P1.27mm -> Package_SO:SO-14_3.9x8.65mm_P1.27mm
- moved REF** 87.7 mm to (101.6, 49.5)
- moved J5 60.5 mm to (110.5, 103.5), turned to 0 degrees
- moved R9 60.1 mm to (133.7, 108.6), turned to 0 degrees
- moved C7 59.8 mm to (124.8, 97.8), turned to 180 degrees
- moved BT1 59.7 mm to (119.4, 119.4), turned to 0 degrees
- moved R6 58.5 mm to (140.2, 63.2)
- moved Y1 54.5 mm to (125.6, 102.2), turned to 90 degrees
- moved TP3 54.2 mm to (94.0, 80.6)
- moved SW1 50.9 mm to (155.0, 92.7), turned to 180 degrees
- moved SW2 50.7 mm to (166.7, 92.7), turned to 180 degrees
- moved SW3 50.7 mm to (178.8, 92.7), turned to 180 degrees
- moved J1 49.9 mm to (165.1, 84.5)
- moved J4 47.6 mm to (165.1, 128.9), turned to -90 degrees
- moved D1 43.5 mm to (134.6, 92.7), turned to 180 degrees
- moved R8 42.1 mm to (133.6, 114.9), turned to 0 degrees
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Connections:
- net /180V renamed /170V
- C1 pad 1: /3.3V_1 -> /5V_1
- C2 pad 1: /3.3V_1 -> /5V_1
- C3 pad 1: /3.3V_1 -> /5V_1
- C4 pad 1: /3.3V_1 -> /5V_1
- C5 pad 1: /3.3V_1 -> /5V_1
- C6 pad 1: Net-(U6-X2) -> GND2
- C6 pad 2: GND2 -> /5V_2
- C7 pad 1: Net-(U6-X1) -> Net-(U8-X2)
- J1 pad 1: /5V_1 -> /DATA
- J1 pad 2: GND1 -> /CLOCK
- J1 pad 3: /12V_1 -> /LATCH
- J2 pad 1: /DATA -> /5V_1
- J2 pad 2: /CLOCK -> GND1
- J2 pad 3: /LATCH -> /12V_1
- J3 pad 1: /HOUR1_EN -> /5V_2
- J3 pad 2: /HOUR2_EN -> GND2
- J3 pad 3: /MINUTE1_EN -> /12V_2
- J4 pad 1: /3.3V_1 -> Net-(J4-Pin_1)
- J4 pad 2: /OE -> Net-(J4-Pin_2)
- J5 pad 1: /5V_2 -> /12V_2
- J5 pad 3: /12V_2 -> GND2
- Q1 pad 1: /HOUR1.0 -> GND1
- R6 pad 2: /HOUR1_EN -> /DOT
- R7 pad 1: Net-(Q11-B) -> /3.3V
- R7 pad 2: /HOUR2_EN -> /SCL
- R8 pad 1: Net-(Q12-B) -> /3.3V
- R8 pad 2: /MINUTE1_EN -> /SDA
- R9 pad 1: Net-(Q13-B) -> /3.3V
- R9 pad 2: /MINUTE2_EN -> /MFP
- SW1 pad 1: /SWITCH.3 -> /SWITCH.1
- SW3 pad 1: /SWITCH.1 -> /SWITCH.3
- U1 pad 1: /HOUR1.1 -> (no net)
- U1 pad 10: unconnected-(U1-~{SRCLR}-Pad10) -> GND1
- U1 pad 11: /CLOCK -> GND1
- U1 pad 13: /OE -> /CLOCK
- U1 pad 14: /DATA -> Net-(U1-DRAIN4)
- U1 pad 15: /HOUR1.0 -> Net-(U1-DRAIN5)
- U1 pad 16: /3.3V_1 -> Net-(U1-DRAIN6)
- U1 pad 2: /HOUR1.2 -> /5V_1
- U1 pad 3: /HOUR1.3 -> /DATA
- U1 pad 4: /HOUR1.4 -> Net-(U1-DRAIN0)
- U1 pad 5: /HOUR1.5 -> Net-(U1-DRAIN1)
- U1 pad 6: /HOUR1.6 -> Net-(U1-DRAIN2)
- U1 pad 7: /HOUR1.7 -> Net-(U1-DRAIN3)
- U1 pad 8: GND1 -> unconnected-(U1-~{SRCLR}-Pad8)
- U1 pad 9: Net-(U1-QH') -> /OE
- U2 pad 1: /HOUR1.9 -> (no net)
- U2 pad 10: unconnected-(U2-~{SRCLR}-Pad10) -> GND1
- U2 pad 11: /CLOCK -> GND1
- U2 pad 13: /OE -> /CLOCK
- U2 pad 14: Net-(U1-QH') -> Net-(U2-DRAIN4)
- U2 pad 15: /HOUR1.8 -> Net-(U2-DRAIN5)
- U2 pad 16: /3.3V_1 -> Net-(U2-DRAIN6)
- U2 pad 2: /HOUR2.0 -> /5V_1
- U2 pad 3: /HOUR2.1 -> Net-(U1-SEROUT)
- U2 pad 4: /HOUR2.2 -> Net-(U2-DRAIN0)
- U2 pad 5: /HOUR2.3 -> Net-(U2-DRAIN1)
- U2 pad 6: /HOUR2.4 -> Net-(U2-DRAIN2)
- U2 pad 7: /HOUR2.5 -> Net-(U2-DRAIN3)
- U2 pad 8: GND1 -> unconnected-(U2-~{SRCLR}-Pad8)
- U2 pad 9: Net-(U2-QH') -> /OE
- U3 pad 1: /HOUR2.7 -> (no net)
- U3 pad 10: unconnected-(U3-~{SRCLR}-Pad10) -> GND1
- U3 pad 11: /CLOCK -> GND1
- U3 pad 13: /OE -> /CLOCK
- U3 pad 14: Net-(U2-QH') -> Net-(U3-DRAIN4)
- U3 pad 15: /HOUR2.6 -> Net-(U3-DRAIN5)
- U3 pad 16: /3.3V_1 -> Net-(U3-DRAIN6)
- U3 pad 2: /HOUR2.8 -> /5V_1
- U3 pad 3: /HOUR2.9 -> Net-(U2-SEROUT)
- U3 pad 4: /MINUTE1.0 -> Net-(U3-DRAIN0)
- U3 pad 5: /MINUTE1.1 -> Net-(U3-DRAIN1)
- U3 pad 6: /MINUTE1.2 -> Net-(U3-DRAIN2)
- U3 pad 7: /MINUTE1.3 -> Net-(U3-DRAIN3)
- U3 pad 8: GND1 -> unconnected-(U3-~{SRCLR}-Pad8)
- U3 pad 9: Net-(U3-QH') -> /OE
- U4 pad 1: /MINUTE1.5 -> (no net)
- U4 pad 10: unconnected-(U4-~{SRCLR}-Pad10) -> GND1
- U4 pad 11: /CLOCK -> GND1
- U4 pad 13: /OE -> /CLOCK
- U4 pad 14: Net-(U3-QH') -> Net-(U4-DRAIN4)
- U4 pad 15: /MINUTE1.4 -> Net-(U4-DRAIN5)
- U4 pad 16: /3.3V_1 -> Net-(U4-DRAIN6)
- U4 pad 2: /MINUTE1.6 -> /5V_1
- U4 pad 3: /MINUTE1.7 -> Net-(U3-SEROUT)
- U4 pad 4: /MINUTE1.8 -> Net-(U4-DRAIN0)
- U4 pad 5: /MINUTE1.9 -> Net-(U4-DRAIN1)
- U4 pad 6: /MINUTE2.0 -> Net-(U4-DRAIN2)
- U4 pad 7: /MINUTE2.1 -> Net-(U4-DRAIN3)
- U4 pad 8: GND1 -> unconnected-(U4-~{SRCLR}-Pad8)
- U4 pad 9: Net-(U4-QH') -> /OE
- U5 pad 1: /MINUTE2.3 -> (no net)
- U5 pad 10: unconnected-(U5-~{SRCLR}-Pad10) -> GND1
- U5 pad 11: /CLOCK -> GND1
- U5 pad 13: /OE -> /CLOCK
- U5 pad 14: Net-(U4-QH') -> Net-(U5-DRAIN4)
- U5 pad 15: /MINUTE2.2 -> Net-(U5-DRAIN5)
- U5 pad 16: /3.3V_1 -> Net-(U5-DRAIN6)
- U5 pad 2: /MINUTE2.4 -> /5V_1
- U5 pad 3: /MINUTE2.5 -> Net-(U4-SEROUT)
- U5 pad 4: /MINUTE2.6 -> Net-(U5-DRAIN0)
- U5 pad 5: /MINUTE2.7 -> Net-(U5-DRAIN1)
- U5 pad 6: /MINUTE2.8 -> Net-(U5-DRAIN2)
- U5 pad 7: /MINUTE2.9 -> Net-(U5-DRAIN3)
- U5 pad 8: GND1 -> unconnected-(U5-~{SRCLR}-Pad8)
- U5 pad 9: unconnected-(U5-QH'-Pad9) -> /OE
- U6 pad 1: Net-(U6-X1) -> GND2
- U6 pad 2: Net-(U6-X2) -> /MCU_OE
- U6 pad 3: Net-(BT1-+) -> Net-(J4-Pin_4)
- U6 pad 5: /SDA -> /MCU_LATCH
- U6 pad 6: /SCL -> Net-(J4-Pin_3)
- U6 pad 7: /MFP -> GND2
- U6 pad 8: /3.3V_2 -> Net-(J4-Pin_2)
- U7 pad 14: /MCU_MINUTE2_EN -> unconnected-(U7-GPIO10-Pad14)
- U7 pad 15: /MCU_MINUTE1_EN -> unconnected-(U7-GPIO11-Pad15)
- U7 pad 16: /MCU_HOUR2_EN -> unconnected-(U7-GPIO12-Pad16)
- U7 pad 17: /MCU_HOUR1_EN -> unconnected-(U7-GPIO13-Pad17)
- U7 pad 19: /MCU_OE -> unconnected-(U7-GPIO14-Pad19)
- U7 pad 36: /3.3V_2 -> /3.3V
- U7 pad 7: unconnected-(U7-GPIO5-Pad7) -> /MCU_OE
- V1 pad 1: Net-(Q6-C) -> Net-(U1-DRAIN1)
- V1 pad 10: Net-(Q1-C) -> Net-(U1-DRAIN0)
- V1 pad 2: Net-(Q10-C) -> Net-(U1-DRAIN2)
- V1 pad 3: Net-(Q14-C) -> Net-(U1-DRAIN3)
- V1 pad 4: Net-(Q18-C) -> Net-(U1-DRAIN4)
- V1 pad 5: Net-(Q22-C) -> Net-(U1-DRAIN5)
- V1 pad 6: Net-(Q26-C) -> Net-(U1-DRAIN6)
- V1 pad 7: Net-(Q30-C) -> Net-(U1-DRAIN7)
- V1 pad 8: Net-(Q34-C) -> Net-(U2-DRAIN0)
- V1 pad 9: Net-(Q38-C) -> Net-(U2-DRAIN1)
- V2 pad 1: Net-(Q7-C) -> Net-(U2-DRAIN3)
- V2 pad 10: Net-(Q2-C) -> Net-(U2-DRAIN2)
- V2 pad 2: Net-(Q11-C) -> Net-(U2-DRAIN4)
- V2 pad 3: Net-(Q15-C) -> Net-(U2-DRAIN5)
- V2 pad 4: Net-(Q19-C) -> Net-(U2-DRAIN6)
- V2 pad 5: Net-(Q23-C) -> Net-(U2-DRAIN7)
- V2 pad 6: Net-(Q27-C) -> Net-(U3-DRAIN0)
- V2 pad 7: Net-(Q31-C) -> Net-(U3-DRAIN1)
- V2 pad 8: Net-(Q35-C) -> Net-(U3-DRAIN2)
- V2 pad 9: Net-(Q39-C) -> Net-(U3-DRAIN3)
- V3 pad 1: Net-(Q8-C) -> Net-(U3-DRAIN5)
- V3 pad 10: Net-(Q3-C) -> Net-(U3-DRAIN4)
- V3 pad 2: Net-(Q12-C) -> Net-(U3-DRAIN6)
- V3 pad 3: Net-(Q16-C) -> Net-(U3-DRAIN7)
- V3 pad 4: Net-(Q20-C) -> Net-(U4-DRAIN0)
- V3 pad 5: Net-(Q24-C) -> Net-(U4-DRAIN1)
- V3 pad 6: Net-(Q28-C) -> Net-(U4-DRAIN2)
- V3 pad 7: Net-(Q32-C) -> Net-(U4-DRAIN3)
- V3 pad 8: Net-(Q36-C) -> Net-(U4-DRAIN4)
- V3 pad 9: Net-(Q40-C) -> Net-(U4-DRAIN5)
- V4 pad 1: Net-(Q9-C) -> Net-(U4-DRAIN7)
- V4 pad 10: Net-(Q4-C) -> Net-(U4-DRAIN6)
- V4 pad 2: Net-(Q13-C) -> Net-(U5-DRAIN0)
- V4 pad 3: Net-(Q17-C) -> Net-(U5-DRAIN1)
- V4 pad 4: Net-(Q21-C) -> Net-(U5-DRAIN2)
- V4 pad 5: Net-(Q25-C) -> Net-(U5-DRAIN3)
- V4 pad 6: Net-(Q29-C) -> Net-(U5-DRAIN4)
- V4 pad 7: Net-(Q33-C) -> Net-(U5-DRAIN5)
- V4 pad 8: Net-(Q37-C) -> Net-(U5-DRAIN6)
- V4 pad 9: Net-(Q41-C) -> Net-(U5-DRAIN7)
- V5 pad C: Net-(Q5-C) -> Net-(Q1-C)
- Y1 pad 1: Net-(U6-X1) -> Net-(U8-X1)
- Y1 pad 2: Net-(U6-X2) -> Net-(U8-X2)
Routing:
- net GND1: track 314.5 -> 94.2 mm, vias 4 -> 5
- net /5V_1: track 108.3 -> 210.2 mm, vias 0 -> 5
- net /3.3V_1: track 94.0 -> 0.00 mm, vias 5 -> 0
- net /3.3V_2: track 88.6 -> 0.00 mm
- net /5V_2: track 5.10 -> 88.9 mm, vias 0 -> 1
- net Net-(Q11-B): track 75.1 -> 0.00 mm
- net Net-(Q13-B): track 75.1 -> 0.00 mm
- net Net-(Q12-B): track 75.1 -> 0.00 mm
- net /3.3V: track 0.00 -> 69.3 mm
- net Net-(Q1-B): track 75.1 -> 7.18 mm
- net /HOUR1_EN: track 61.0 -> 0.00 mm
- net /MINUTE2.0: track 51.1 -> 0.00 mm
- net /MINUTE2.9: track 47.4 -> 0.00 mm
- net /MINUTE2_EN: track 42.6 -> 0.00 mm
- net /MINUTE1.0: track 42.2 -> 0.00 mm
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- added copper zone on B.Cu, net GND1
- removed copper zone on B.Cu, net (none)
Other:
- board size 116.8 x 91.4 mm -> 113 x 86.4 mm
