File: kicad/Nixie IN-8.kicad_pcb (KiCad board)
At the start: 2 copper layers, 113 x 86.4 mm, 57 parts, among them J1 Conn_01x05_Pin, J2 Conn_01x03_Pin, J3 Conn_01x03_Pin, J4 Conn_01x05_Pin, J5 Barrel_Jack_Switch, Q1 MPSA42, SW1 SW_SPST, SW2 SW_SPST, SW3 SW_SPST, U1 TPIC6B595, U2 TPIC6B595, U3 TPIC6B595, U4 TPIC6B595, U5 TPIC6B595, U6 SN74AHCT125, U7 Pico, U8 MCP7940N-xP, Y1 32.768kHz

Commit message: finished pcb
Parts:
- removed the REF** at (186.7, 127.0)
- removed the REF** at (186.7, 94.0)
- removed the mouse-bite-2.54mm-slot at (186.1, 88.3)
- R1, R2, R3, R4: value 8.66k -> 10k
- moved mouse-bite-2.54mm-slot 26.9 mm to (179.3, 88.3)
- moved mouse-bite-2.54mm-slot 9.73 mm to (109.0, 88.3)
- moved J5 1.27 mm to (110.5, 102.2)
- moved SW1 0.58 mm to (155.0, 92.1)
- moved SW2 0.58 mm to (166.7, 92.1)
- moved SW3 0.58 mm to (178.8, 92.1)
Routing:
- net GND2: track 66.3 -> 70.9 mm
- net /5V_2: track 88.9 -> 91.1 mm
- net Net-(U3-DRAIN0): track 29.1 -> 31.0 mm
- net Net-(U1-DRAIN1): track 28.7 -> 30.5 mm
- net Net-(D1-K): track 57.6 -> 59.1 mm
- net /SWITCH.2: track 11.6 -> 12.8 mm
- net Net-(U1-DRAIN2): track 29.1 -> 30.3 mm
- net /12V_2: track 19.2 -> 18.3 mm
- net /5V_1: track 210.2 -> 211.1 mm
- net /170V: track 127.6 -> 126.8 mm
- net /SWITCH.3: track 10.9 -> 11.4 mm
Other:
- board size 113 x 86.4 mm -> 113 x 88.3 mm
