File: kicad/Nixie IN-8.kicad_sch (KiCad schematic)
At the start: 93 parts, among them J1 Conn_01x03_Pin, J2 Conn_01x04_Pin, J3 Conn_01x04_Pin, J4 Conn_01x02_Pin, J5 Conn_01x03_Pin, J6 Conn_01x04_Pin, J7 Conn_01x04_Pin, J8 Conn_01x02_Pin, J9 Barrel_Jack_Switch, Q1 MPSA42, Q10 MPSA42, Q11 MPSA42, Q12 MPSA42, Q13 MPSA42, Q14 MPSA42, Q15 MPSA42, Q16 MPSA42, Q17 MPSA42, Q18 MPSA42, Q19 MPSA42, Q2 MPSA42, Q20 MPSA42, Q21 MPSA42, Q22 MPSA42, Q23 MPSA42, Q24 MPSA42, Q25 MPSA42, Q26 MPSA42, Q27 MPSA42, Q28 MPSA42, Q29 MPSA42, Q3 MPSA42, Q30 MPSA42, Q31 MPSA42, Q32 MPSA42, Q33 MPSA42, Q34 MPSA42, Q35 MPSA42, Q36 MPSA42, Q37 MPSA42, Q38 MPSA42, Q39 MPSA42, Q4 MPSA42, Q40 MPSA42, Q41 MPSA42, Q5 MPSA42, Q6 MPSA42, Q7 MPSA42, Q8 MPSA42, Q9 MPSA42, SW1 SW_SPST, SW2 SW_SPST, SW3 SW_SPST, U1 74HC595, U2 74HC595, U3 74HC595, U4 74HC595, U5 74HC595, U6 MCP7940N-xP, U7 Pico, Y1 32.768kHz

Commit message: finished routing
Parts:
- removed J2, J3, J6, J7: Conn_01x04_Pin, Connector_PinHeader_2.54mm:PinHeader_1x04_P2.54mm_Vertical, symbol Connector:Conn_01x04_Pin
- removed J4, J8: Conn_01x02_Pin, Connector_PinHeader_2.54mm:PinHeader_1x02_P2.54mm_Vertical, symbol Connector:Conn_01x02_Pin
- removed Q1, Q10, Q11, Q12, Q13, Q14, Q15, Q16, Q17, Q18, Q19, Q2, Q20, Q21, Q22, Q23, Q24, Q25, Q26, Q27, Q28, Q29, Q3, Q30, Q31, Q32, Q33, Q34, Q35, Q36, Q37, Q38, Q39, Q4, Q40, Q41, Q6, Q7, Q8, Q9: MPSA42, Package_TO_SOT_THT:TO-92_Inline_Wide, symbol Nixie:NPN-MPSA42
- removed R6, R7, R8, R9: 13.5k, Resistor_THT:R_Axial_DIN0204_L3.6mm_D1.6mm_P5.08mm_Vertical, symbol Device:R
- removed U1, U2, U3, U4, U5: 74HC595, Package_SO:SOIC-16_3.9x9.9mm_P1.27mm, symbol 74xx:74HC595
- added C6, C9: 0.1µF, Capacitor_SMD:C_1206_3216Metric_Pad1.33x1.80mm_HandSolder, symbol Device:C
- added J1, J4: Conn_01x05_Pin, Connector_PinHeader_2.54mm:PinHeader_1x05_P2.54mm_Vertical, symbol Connector:Conn_01x05_Pin
- added U1, U2, U3, U4, U5: TPIC6B595, Package_SO:SOIC-20W_7.5x12.8mm_P1.27mm, symbol Nixie:TPIC6B595
- added U6: SN74AHCT125, Package_SO:SO-14_3.9x8.65mm_P1.27mm, symbol Nixie:SN54AHCT125
- R1, R2, R3, R4: value 12k -> 8.66k
- R5: value 200k -> 162k
- R6: renamed from R10; footprint Resistor_THT:R_Axial_DIN0204_L3.6mm_D1.6mm_P5.08mm_Vertical -> Resistor_THT:R_Axial_DIN0204_L3.6mm_D1.6mm_P5.08mm_Horizontal
- TP1: value 180V -> 170V
- renumbered C6 to C7, C7 to C8, J1 to J2, J5 to J3, J9 to J5, Q5 to Q1, R11 to R7, R12 to R8, R13 to R9, SW3 to SW1, SW1 to SW3, U6 to U8
Connections:
- net 3.3V_1 is gone; now on net 5V_1: C1.1, C2.1, C3.1, C4.1, C5.1
- net 5V_1: now also U1.2 (VCC), U2.2 (VCC), U3.2 (VCC), U4.2 (VCC), U5.2 (VCC)
- net 5V_2: now also C6.2, U6.14 (VCC)
- net CLOCK: now also J1.2 (Pin_2), U1.13 (SRCK), U2.13 (SRCK), U3.13 (SRCK), U4.13 (SRCK), U5.13 (SRCK)
- net DATA: now also J1.1 (Pin_1), U1.3 (SERIN)
- net DOT: now also J1.5 (Pin_5)
- net GND1: now also U1.10 (GND), U1.11 (GND), U1.19 (GND), U2.10 (GND), U2.11 (GND), U2.19 (GND), U3.10 (GND), U3.11 (GND), U3.19 (GND), U4.10 (GND), U4.11 (GND), U4.19 (GND), U5.10 (GND), U5.11 (GND), U5.19 (GND)
- net GND2: now also C6.1, C9.2, U6.1 (~{1OE}), U6.10 (~{3OE}), U6.13 (~{4OE}), U6.4 (~{2OE}), U6.7 (GND)
- net LATCH: now also J1.3 (Pin_3), U1.12 (RCK), U2.12 (RCK), U3.12 (RCK), U4.12 (RCK), U5.12 (RCK)
- net MCU_CLOCK: now also U6.9 (3A)
- net MCU_DATA: now also U6.12 (4A)
- net MCU_DOT: now also J4.5 (Pin_5)
- net MCU_LATCH: now also U6.5 (2A)
- net MCU_OE: now also U7.7 (GPIO5), U6.2 (1A); no longer U7.19 (GPIO14)
- net OE: now also J1.4 (Pin_4), U1.9 (~{G}), U2.9 (~{G}), U3.9 (~{G}), U4.9 (~{G}), U5.9 (~{G})
- net at V1.8: now also U2.4 (DRAIN0)
- net at V2.1: now also U2.7 (DRAIN3)
- net at V1.7: now also U1.17 (DRAIN7)
- net at V3.1: now also U3.15 (DRAIN5)
- net at V1.4: now also U1.14 (DRAIN4)
- net at V2.5: now also U2.17 (DRAIN7)
- net at V4.8: now also U5.16 (DRAIN6)
- net at V2.8: now also U3.6 (DRAIN2)
- net at V1.9: now also U2.5 (DRAIN1)
- net at V4.1: now also U4.17 (DRAIN7)
- net at V4.10 (0): now also U4.16 (DRAIN6)
- net at V4.2: now also U5.4 (DRAIN0)
- net at V4.3: now also U5.5 (DRAIN1)
- net at V4.4: now also U5.6 (DRAIN2)
- net at V4.5: now also U5.7 (DRAIN3)
- net at V4.6: now also U5.14 (DRAIN4)
- net at V4.7: now also U5.15 (DRAIN5)
- net at V4.9: now also U5.17 (DRAIN7)
- net at V3.5: now also U4.5 (DRAIN1)
- net at V1.1: now also U1.5 (DRAIN1)
- net at V3.10 (0): now also U3.14 (DRAIN4)
- net at V3.2: now also U3.16 (DRAIN6)
- net at V3.3: now also U3.17 (DRAIN7)
- net at V3.4: now also U4.4 (DRAIN0)
- net at V3.6: now also U4.6 (DRAIN2)
- net at V3.7: now also U4.7 (DRAIN3)
- net at V3.8: now also U4.14 (DRAIN4)
- net at V3.9: now also U4.15 (DRAIN5)
- net at V2.10 (0): now also U2.6 (DRAIN2)
- net at V2.6: now also U3.4 (DRAIN0)
- net at V2.9: now also U3.7 (DRAIN3)
- net at V2.7: now also U3.5 (DRAIN1)
- net at V1.5: now also U1.15 (DRAIN5)
- net at V2.3: now also U2.15 (DRAIN5)
- net at V1.6: now also U1.16 (DRAIN6)
- net at V2.2: now also U2.14 (DRAIN4)
- net at V2.4: now also U2.16 (DRAIN6)
- net at V1.10 (0): now also U1.4 (DRAIN0)
- net at V1.2: now also U1.6 (DRAIN2)
- net at V1.3: now also U1.7 (DRAIN3)
- net 180V renamed 170V
- net 3.3V_2 renamed 3.3V
- net 3.3V: now also C9.1
- net MCU_HOUR1_EN: no longer names the net of U7.17 (GPIO13)
- net MCU_HOUR2_EN: no longer names the net of U7.16 (GPIO12)
- net MCU_MINUTE1_EN: no longer names the net of U7.15 (GPIO11)
- net MCU_MINUTE2_EN: no longer names the net of U7.14 (GPIO10)
- new net: U3.18 (SEROUT), U4.3 (SERIN)
- new net: U2.18 (SEROUT), U3.3 (SERIN)
- new net: U4.18 (SEROUT), U5.3 (SERIN)
- new net: J4.1 (Pin_1), U6.11 (4Y)
- new net: J4.2 (Pin_2), U6.8 (3Y)
- new net: J4.3 (Pin_3), U6.6 (2Y)
- new net: J4.4 (Pin_4), U6.3 (1Y)
- new net: U1.18 (SEROUT), U2.3 (SERIN)
Other:
- note added: "Anode Volate 150V Rated Current 2.5mA Max Current 3.5mA"
- note added: "Anode Volate 70V Rated Current 0.6mA Max Current 1mA"
- note removed: "SHIFT REGISTERS"
- note removed: "TUBES"
- moved on the sheet: BT1, C7, C8, D1, J2, J3, J5, Q1, R1, R2, R3, R4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

Commit message: finished pcb
Parts:
- R1, R2, R3, R4: value 8.66k -> 10k
Changed lines of the file:
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@@
       (effects (font (size 1.27 1.27)) (justify left))
     )
-    (property "Value" "8.66k" (at 109.22 38.1 0)
+    (property "Value" "10k" (at 109.22 38.1 0)
       (effects (font (size 1.27 1.27)) (justify left))
     )
@@
       (effects (font (size 1.27 1.27)) (justify left))
     )
-    (property "Value" "8.66k" (at 213.36 38.1 0)
+    (property "Value" "10k" (at 213.36 38.1 0)
       (effects (font (size 1.27 1.27)) (justify left))
     )
@@
       (effects (font (size 1.27 1.27)) (justify left))
     )
-    (property "Value" "8.66k" (at 161.29 38.1 0)
+    (property "Value" "10k" (at 161.29 38.1 0)
       (effects (font (size 1.27 1.27)) (justify left))
     )
@@
       (effects (font (size 1.27 1.27)) (justify left))
     )
-    (property "Value" "8.66k" (at 57.15 38.1 0)
-      (effects (font (size 1.27 1.27)) (justify left))
-    )
+    (property "Value" "10k" (at 57.15 38.1 0)
+      (effects (font (size 1.27 1.27)) (justify left))
+    )
